File: PCB/HeManTCN/CPU.sch (KiCad schematic (older format))
At the start: 24 parts

Commit message: Hoja A1
Desarme las hojas jerarquicas y configure la hoja del esquematico como A1. Hay lugar suficiente (por ahora) para todo.
Parts:
- gave numbers to parts that had none: 24
