File: PCB/HeManTCN/Debug-Serial.sch (KiCad schematic (older format))
At the start: 6 parts

Commit message: Hoja A1
Desarme las hojas jerarquicas y configure la hoja del esquematico como A1. Hay lugar suficiente (por ahora) para todo.
Parts:
- gave numbers to parts that had none: 6
Changed lines of the file:
@@
 $Descr A4 11693 8268
 encoding utf-8
-Sheet 11 11
+Sheet 11 8
 Title "SnifferTCN"
 Date "2019-09-25"
@@
 U 1 1 5DA601E1
 P 5900 4400
-F 0 "#PWR?" H 5900 4150 50  0001 C CNN
+AR Path="/5DA601E1" Ref="#PWR?"  Part="1"
+AR Path="/5DA600DB/5DA601E1" Ref="#PWR01107"  Part="1"
+F 0 "#PWR01107" H 5900 4150 50  0001 C CNN
 F 1 "GND" H 5905 4227 50  0000 C CNN
 F 2 "" H 5900 4400 50  0001 C CNN
@@
 U 1 1 5DA601E7
 P 4850 3100
-F 0 "#PWR?" H 4850 2850 50  0001 C CNN
+AR Path="/5DA601E7" Ref="#PWR?"  Part="1"
+AR Path="/5DA600DB/5DA601E7" Ref="#PWR01104"  Part="1"
+F 0 "#PWR01104" H 4850 2850 50  0001 C CNN
 F 1 "GND" V 4855 2972 50  0000 R CNN
 F 2 "" H 4850 3100 50  0001 C CNN
@@
 U 1 1 5DA601F1
 P 6000 2900
-F 0 "#PWR?" H 6000 2750 50  0001 C CNN
+AR Path="/5DA601F1" Ref="#PWR?"  Part="1"
+AR Path="/5DA600DB/5DA601F1" Ref="#PWR01108"  Part="1"
+F 0 "#PWR01108" H 6000 2750 50  0001 C CNN
 F 1 "+3.3V" V 6015 3028 50  0000 L CNN
 F 2 "" H 6000 2900 50  0001 C CNN
@@
 U 1 1 5DA601F8
 P 4950 3100
-F 0 "C?" V 4813 3100 50  0000 C CNN
+AR Path="/5DA601F8" Ref="C?"  Part="1"
+AR Path="/5DA600DB/5DA601F8" Ref="C1101"  Part="1"
+F 0 "C1101" V 4813 3100 50  0000 C CNN
 F 1 "0.1u" V 4722 3100 50  0000 C CNN
 F 2 "Capacitor_SMD:C_0805_2012Metric" H 4950 3100 50  0001 C CNN
@@
 U 1 1 5DA6020F
 P 6100 3600
-F 0 "U?" H 6450 2850 50  0000 C CNN
+AR Path="/5DA6020F" Ref="U?"  Part="1"
+AR Path="/5DA600DB/5DA6020F" Ref="U1101"  Part="1"
+F 0 "U1101" H 6450 2850 50  0000 C CNN
 F 1 "STM32F042F6Px" H 6550 2750 50  0000 C CNN
 F 2 "Package_SO:TSSOP-20_4.4x6.5mm_P0.65mm" H 5600 2900 50  0001 R CNN
@@
 U 1 1 5DA60222
 P 4450 3700
-F 0 "#PWR?" H 4450 3450 50  0001 C CNN
+AR Path="/5DA60222" Ref="#PWR?"  Part="1"
+AR Path="/5DA600DB/5DA60222" Ref="#PWR01103"  Part="1"
+F 0 "#PWR01103" H 4450 3450 50  0001 C CNN
 F 1 "GND" V 4455 3572 50  0000 R CNN
 F 2 "" H 4450 3700 50  0001 C CNN
@@
 U 1 1 5DA60229
 P 4750 3700
-F 0 "J?" H 4800 3800 50  0000 C CNN
+AR Path="/5DA60229" Ref="J?"  Part="1"
+AR Path="/5DA600DB/5DA60229" Ref="J1102"  Part="1"
+F 0 "J1102" H 4800 3800 50  0000 C CNN
 F 1 "Conn_02x02_Odd_Even" H 4700 3500 50  0000 C CNN
 F 2 "Pin_Headers:Pin_Header_Straight_2x02_Pitch2.54mm" H 4750 3700 50  0001 C CNN
@@
 U 1 1 5DA60231
 P 5050 4200
-F 0 "R?" V 4946 4200 50  0000 C CNN
+AR Path="/5DA60231" Ref="R?"  Part="1"
+AR Path="/5DA600DB/5DA60231" Ref="R1101"  Part="1"
+F 0 "R1101" V 4946 4200 50  0000 C CNN
 F 1 "4K7" V 4855 4200 50  0000 C CNN
 F 2 "Resistor_SMD:R_0805_2012Metric" H 5050 4200 50  0001 C CNN
@@
 U 1 1 5DA60238
 P 4950 4200
-F 0 "#PWR?" H 4950 3950 50  0001 C CNN
+AR Path="/5DA60238" Ref="#PWR?"  Part="1"
+AR Path="/5DA600DB/5DA60238" Ref="#PWR01105"  Part="1"
+F 0 "#PWR01105" H 4950 3950 50  0001 C CNN
 F 1 "GND" V 4955 4072 50  0000 R CNN
 F 2 "" H 4950 4200 50  0001 C CNN
@@
 U 1 1 5DA6023E
 P 4650 2750
-F 0 "J?" H 4700 3067 50  0000 C CNN
+AR Path="/5DA6023E" Ref="J?"  Part="1"
+AR Path="/5DA600DB/5DA6023E" Ref="J1101"  Part="1"
+F 0 "J1101" H 4700 3067 50  0000 C CNN
 F 1 "Conn_02x03_Odd_Even" H 4700 2976 50  0000 C CNN
 F 2 "Connector_PinHeader_2.54mm:PinHeader_2x03_P2.54mm_Vertical" H 4650 2750 50  0001 C CNN
@@
 U 1 1 5DA60245
 P 4150 2650
-F 0 "#PWR?" H 4150 2500 50  0001 C CNN
+AR Path="/5DA60245" Ref="#PWR?"  Part="1"
+AR Path="/5DA600DB/5DA60245" Ref="#PWR01101"  Part="1"
+F 0 "#PWR01101" H 4150 2500 50  0001 C CNN
 F 1 "+3.3V" V 4165 2778 50  0000 L CNN
 F 2 "" H 4150 2650 50  0001 C CNN
@@
 U 1 1 5DA60251
 P 5550 2900
-F 0 "#PWR?" H 5550 2650 50  0001 C CNN
+AR Path="/5DA60251" Ref="#PWR?"  Part="1"
+AR Path="/5DA600DB/5DA60251" Ref="#PWR01106"  Part="1"
+F 0 "#PWR01106" H 5550 2650 50  0001 C CNN
 F 1 "GND" V 5555 2772 50  0000 R CNN
 F 2 "" H 5550 2900 50  0001 C CNN
@@
 U 1 1 5DA60257
 P 4150 2750
-F 0 "#PWR?" H 4150 2500 50  0001 C CNN
+AR Path="/5DA60257" Ref="#PWR?"  Part="1"
+AR Path="/5DA600DB/5DA60257" Ref="#PWR01102"  Part="1"
+F 0 "#PWR01102" H 4150 2500 50  0001 C CNN
 F 1 "GND" V 4155 2622 50  0000 R CNN
 F 2 "" H 4150 2750 50  0001 C CNN
@@
 U 1 1 5DA60263
 P 5650 2900
-F 0 "C?" V 5879 2900 50  0000 C CNN
+AR Path="/5DA60263" Ref="C?"  Part="1"
+AR Path="/5DA600DB/5DA60263" Ref="C1102"  Part="1"
+F 0 "C1102" V 5879 2900 50  0000 C CNN
 F 1 "0.1u" V 5788 2900 50  0000 C CNN
 F 2 "Capacitor_SMD:C_0805_2012Metric" H 5650 2900 50  0001 C CNN
