File: PCB/HeManTCN/Ethernet.sch (KiCad schematic (older format))
At the start: 18 parts

Commit message: Hoja A1
Desarme las hojas jerarquicas y configure la hoja del esquematico como A1. Hay lugar suficiente (por ahora) para todo.
Parts:
- gave numbers to parts that had none: 18
Changed lines of the file:
@@
 $Descr A4 11693 8268
 encoding utf-8
-Sheet 7 11
+Sheet 7 3
 Title "SnifferTCN"
 Date "2019-09-25"
@@
 U 1 1 5DA5A9DB
 P 4350 3500
-F 0 "U?" H 3800 4550 50  0000 C CNN
+AR Path="/5DA5A9DB" Ref="U?"  Part="1"
+AR Path="/5DA5A719/5DA5A9DB" Ref="U701"  Part="1"
+F 0 "U701" H 3800 4550 50  0000 C CNN
 F 1 "KSZ8081RNA" H 4800 4550 50  0000 C CNN
 F 2 "Package_DFN_QFN:QFN-24-1EP_4x4mm_P0.5mm_EP2.6x2.6mm" H 5750 2500 50  0001 C CNN
@@
 U 1 1 5DA5A9E2
 P 4350 4500
-F 0 "#PWR?" H 4350 4250 50  0001 C CNN
+AR Path="/5DA5A9E2" Ref="#PWR?"  Part="1"
+AR Path="/5DA5A719/5DA5A9E2" Ref="#PWR0705"  Part="1"
+F 0 "#PWR0705" H 4350 4250 50  0001 C CNN
 F 1 "GND" V 4355 4372 50  0000 R CNN
 F 2 "" H 4350 4500 50  0001 C CNN
@@
 U 1 1 5DA5A9ED
 P 3650 2250
-F 0 "C?" H 3742 2296 50  0000 L CNN
+AR Path="/5DA5A9ED" Ref="C?"  Part="1"
+AR Path="/5DA5A719/5DA5A9ED" Ref="C704"  Part="1"
+F 0 "C704" H 3742 2296 50  0000 L CNN
 F 1 "2.2u" H 3742 2205 50  0000 L CNN
 F 2 "Capacitor_SMD:C_0805_2012Metric" H 3650 2250 50  0001 C CNN
@@
 U 1 1 5DA5A9F5
 P 3950 2250
-F 0 "C?" H 4042 2296 50  0000 L CNN
+AR Path="/5DA5A9F5" Ref="C?"  Part="1"
+AR Path="/5DA5A719/5DA5A9F5" Ref="C705"  Part="1"
+F 0 "C705" H 4042 2296 50  0000 L CNN
 F 1 "4.7u" H 4042 2205 50  0000 L CNN
 F 2 "Capacitor_SMD:C_0805_2012Metric" H 3950 2250 50  0001 C CNN
@@
 U 1 1 5DA5AA02
 P 3550 2350
-F 0 "#PWR?" H 3550 2100 50  0001 C CNN
+AR Path="/5DA5AA02" Ref="#PWR?"  Part="1"
+AR Path="/5DA5A719/5DA5AA02" Ref="#PWR0704"  Part="1"
+F 0 "#PWR0704" H 3550 2100 50  0001 C CNN
 F 1 "GND" V 3555 2222 50  0000 R CNN
 F 2 "" H 3550 2350 50  0001 C CNN
@@
 U 1 1 5DA5AA09
 P 4550 2250
-F 0 "C?" H 4642 2296 50  0000 L CNN
+AR Path="/5DA5AA09" Ref="C?"  Part="1"
+AR Path="/5DA5A719/5DA5AA09" Ref="C706"  Part="1"
+F 0 "C706" H 4642 2296 50  0000 L CNN
 F 1 "4.7u" H 4642 2205 50  0000 L CNN
 F 2 "Capacitor_SMD:C_0805_2012Metric" H 4550 2250 50  0001 C CNN
@@
 U 1 1 5DA5AA11
 P 4850 2250
-F 0 "C?" H 4942 2296 50  0000 L CNN
+AR Path="/5DA5AA11" Ref="C?"  Part="1"
+AR Path="/5DA5A719/5DA5AA11" Ref="C707"  Part="1"
+F 0 "C707" H 4942 2296 50  0000 L CNN
 F 1 "0.1u" H 4942 2205 50  0000 L CNN
 F 2 "Capacitor_SMD:C_0805_2012Metric" H 4850 2250 50  0001 C CNN
@@
 U 1 1 5DA5AA19
 P 5150 2250
-F 0 "C?" H 5242 2296 50  0000 L CNN
+AR Path="/5DA5AA19" Ref="C?"  Part="1"
+AR Path="/5DA5A719/5DA5AA19" Ref="C708"  Part="1"
+F 0 "C708" H 5242 2296 50  0000 L CNN
 F 1 "0.1u" H 5242 2205 50  0000 L CNN
 F 2 "Capacitor_SMD:C_0805_2012Metric" H 5150 2250 50  0001 C CNN
@@
 U 1 1 5DA5AA2D
 P 4450 2050
-F 0 "#PWR?" H 4450 1900 50  0001 C CNN
+AR Path="/5DA5AA2D" Ref="#PWR?"  Part="1"
+AR Path="/5DA5A719/5DA5AA2D" Ref="#PWR0706"  Part="1"
+F 0 "#PWR0706" H 4450 1900 50  0001 C CNN
 F 1 "+3.3V" V 4465 2178 50  0000 L CNN
 F 2 "" H 4450 2050 50  0001 C CNN
@@
 U 1 1 5DA5AA34
 P 5050 4000
-F 0 "R?" H 5109 4046 50  0000 L CNN
+AR Path="/5DA5AA34" Ref="R?"  Part="1"
+AR Path="/5DA5A719/5DA5AA34" Ref="R704"  Part="1"
+F 0 "R704" H 5109 4046 50  0000 L CNN
 F 1 "6.49K 1%" H 5109 3955 50  0000 L CNN
 F 2 "Resistor_SMD:R_0805_2012Metric" H 5050 4000 50  0001 C CNN
@@
 U 1 1 5DA5AA3B
 P 5050 4100
-F 0 "#PWR?" H 5050 3850 50  0001 C CNN
+AR Path="/5DA5AA3B" Ref="#PWR?"  Part="1"
+AR Path="/5DA5A719/5DA5AA3B" Ref="#PWR0707"  Part="1"
+F 0 "#PWR0707" H 5050 3850 50  0001 C CNN
 F 1 "GND" V 5055 3972 50  0000 R CNN
 F 2 "" H 5050 4100 50  0001 C CNN
@@
 U 1 1 5DA5AA48
 P 3100 4000
-F 0 "C?" V 3050 4050 50  0000 L CNN
+AR Path="/5DA5AA48" Ref="C?"  Part="1"
+AR Path="/5DA5A719/5DA5AA48" Ref="C701"  Part="1"
+F 0 "C701" V 3050 4050 50  0000 L CNN
 F 1 "0.1u" V 3150 4050 50  0000 L CNN
 F 2 "Capacitor_SMD:C_0805_2012Metric" H 3100 4000 50  0001 C CNN
@@
 U 1 1 5DA5AA50
 P 3100 3850
-F 0 "R?" V 3100 3500 50  0000 C CNN
+AR Path="/5DA5AA50" Ref="R?"  Part="1"
+AR Path="/5DA5A719/5DA5AA50" Ref="R703"  Part="1"
+F 0 "R703" V 3100 3500 50  0000 C CNN
 F 1 "4K7" V 3100 3650 50  0000 C CNN
 F 2 "Resistor_SMD:R_0805_2012Metric" H 3100 3850 50  0001 C CNN
@@
 U 1 1 5DA5AA58
 P 3100 3700
-F 0 "R?" V 3100 3350 50  0000 C CNN
+AR Path="/5DA5AA58" Ref="R?"  Part="1"
+AR Path="/5DA5A719/5DA5AA58" Ref="R702"  Part="1"
+F 0 "R702" V 3100 3350 50  0000 C CNN
 F 1 "4K7" V 3100 3500 50  0000 C CNN
 F 2 "Resistor_SMD:R_0805_2012Metric" H 3100 3700 50  0001 C CNN
@@
 U 1 1 5DA5AA60
 P 3100 3600
-F 0 "R?" V 3100 3250 50  0000 C CNN
+AR Path="/5DA5AA60" Ref="R?"  Part="1"
+AR Path="/5DA5A719/5DA5AA60" Ref="R701"  Part="1"
+F 0 "R701" V 3100 3250 50  0000 C CNN
 F 1 "4K7" V 3100 3400 50  0000 C CNN
 F 2 "Resistor_SMD:R_0805_2012Metric" H 3100 3600 50  0001 C CNN
@@
 U 1 1 5DA5AA6B
 P 3000 3400
-F 0 "#PWR?" H 3000 3250 50  0001 C CNN
+AR Path="/5DA5AA6B" Ref="#PWR?"  Part="1"
+AR Path="/5DA5A719/5DA5AA6B" Ref="#PWR0701"  Part="1"
+F 0 "#PWR0701" H 3000 3250 50  0001 C CNN
 F 1 "+3.3V" V 3015 3528 50  0000 L CNN
 F 2 "" H 3000 3400 50  0001 C CNN
@@
 U 1 1 5DA5AA71
 P 3000 4000
-F 0 "#PWR?" H 3000 3750 50  0001 C CNN
+AR Path="/5DA5AA71" Ref="#PWR?"  Part="1"
+AR Path="/5DA5A719/5DA5AA71" Ref="#PWR0702"  Part="1"
+F 0 "#PWR0702" H 3000 3750 50  0001 C CNN
 F 1 "GND" H 3005 3827 50  0000 C CNN
 F 2 "" H 3000 4000 50  0001 C CNN
@@
 U 1 1 5DA5AA7D
 P 3250 4500
-F 0 "Y?" H 3250 4275 50  0000 C CNN
+AR Path="/5DA5AA7D" Ref="Y?"  Part="1"
+AR Path="/5DA5A719/5DA5AA7D" Ref="Y701"  Part="1"
+F 0 "Y701" H 3250 4275 50  0000 C CNN
 F 1 "25MHz" H 3250 4366 50  0000 C CNN
 F 2 "Crystal:Crystal_SMD_5032-2Pin_5.0x3.2mm" H 3250 4500 50  0001 C CNN
@@
 U 1 1 5DA5AA85
 P 3100 4600
-F 0 "C?" H 3191 4646 50  0000 L CNN
+AR Path="/5DA5AA85" Ref="C?"  Part="1"
+AR Path="/5DA5A719/5DA5AA85" Ref="C702"  Part="1"
+F 0 "C702" H 3191 4646 50  0000 L CNN
 F 1 "22p" H 3191 4555 50  0000 L CNN
 F 2 "Capacitor_SMD:C_0805_2012Metric" H 3100 4600 50  0001 C CNN
@@
 U 1 1 5DA5AA8D
 P 3400 4600
-F 0 "C?" H 3308 4646 50  0000 R CNN
+AR Path="/5DA5AA8D" Ref="C?"  Part="1"
+AR Path="/5DA5A719/5DA5AA8D" Ref="C703"  Part="1"
+F 0 "C703" H 3308 4646 50  0000 R CNN
 F 1 "22p" H 3308 4555 50  0000 R CNN
 F 2 "Capacitor_SMD:C_0805_2012Metric" H 3400 4600 50  0001 C CNN
@@
 U 1 1 5DA5AA94
 P 3250 4700
-F 0 "#PWR?" H 3250 4450 50  0001 C CNN
+AR Path="/5DA5AA94" Ref="#PWR?"  Part="1"
+AR Path="/5DA5A719/5DA5AA94" Ref="#PWR0703"  Part="1"
+F 0 "#PWR0703" H 3250 4450 50  0001 C CNN
 F 1 "GND" H 3255 4527 50  0000 C CNN
 F 2 "" H 3250 4700 50  0001 C CNN
@@
 U 1 1 5DA5AAA3
 P 5750 3300
-F 0 "C?" V 5521 3300 50  0000 C CNN
+AR Path="/5DA5AAA3" Ref="C?"  Part="1"
+AR Path="/5DA5A719/5DA5AAA3" Ref="C709"  Part="1"
+F 0 "C709" V 5521 3300 50  0000 C CNN
 F 1 "0.1u" V 5612 3300 50  0000 C CNN
 F 2 "Capacitor_SMD:C_0805_2012Metric" H 5750 3300 50  0001 C CNN
@@
 U 1 1 5DA5AAAA
 P 5650 3450
-F 0 "#PWR?" H 5650 3200 50  0001 C CNN
+AR Path="/5DA5AAAA" Ref="#PWR?"  Part="1"
+AR Path="/5DA5A719/5DA5AAAA" Ref="#PWR0708"  Part="1"
+F 0 "#PWR0708" H 5650 3200 50  0001 C CNN
 F 1 "GND" V 5655 3322 50  0000 R CNN
 F 2 "" H 5650 3450 50  0001 C CNN
@@
 U 1 1 5DA5AAB1
 P 5750 3600
-F 0 "C?" V 5887 3600 50  0000 C CNN
+AR Path="/5DA5AAB1" Ref="C?"  Part="1"
+AR Path="/5DA5A719/5DA5AAB1" Ref="C710"  Part="1"
+F 0 "C710" V 5887 3600 50  0000 C CNN
 F 1 "0.1u" V 5978 3600 50  0000 C CNN
 F 2 "Capacitor_SMD:C_0805_2012Metric" H 5750 3600 50  0001 C CNN
@@
 U 1 1 5DA5AABA
 P 6950 4400
-F 0 "#PWR?" H 6950 4150 50  0001 C CNN
+AR Path="/5DA5AABA" Ref="#PWR?"  Part="1"
+AR Path="/5DA5A719/5DA5AABA" Ref="#PWR0710"  Part="1"
+F 0 "#PWR0710" H 6950 4150 50  0001 C CNN
 F 1 "GND" V 6827 4363 50  0000 C CNN
 F 2 "" H 6950 4400 50  0001 C CNN
@@
 U 1 1 5DA5AAC0
 P 7850 4100
-F 0 "#PWR?" H 7850 3850 50  0001 C CNN
+AR Path="/5DA5AAC0" Ref="#PWR?"  Part="1"
+AR Path="/5DA5A719/5DA5AAC0" Ref="#PWR0711"  Part="1"
+F 0 "#PWR0711" H 7850 3850 50  0001 C CNN
 F 1 "GND" H 7800 3950 50  0000 L CNN
 F 2 "" H 7850 4100 50  0001 C CNN
@@
 U 1 1 5DA5AAC7
 P 5650 4200
-F 0 "R?" V 5600 4350 50  0000 C CNN
+AR Path="/5DA5AAC7" Ref="R?"  Part="1"
+AR Path="/5DA5A719/5DA5AAC7" Ref="R705"  Part="1"
+F 0 "R705" V 5600 4350 50  0000 C CNN
 F 1 "220R" V 5700 4400 50  0000 C CNN
 F 2 "Resistor_SMD:R_0805_2012Metric" H 5650 4200 50  0001 C CNN
@@
 U 1 1 5DA5AAD6
 P 6950 3700
-F 0 "J?" H 6950 4425 50  0000 C CNN
+AR Path="/5DA5AAD6" Ref="J?"  Part="1"
+AR Path="/5DA5A719/5DA5AAD6" Ref="J701"  Part="1"
+F 0 "J701" H 6950 4425 50  0000 C CNN
 F 1 "RJ45_Amphenol_RJMG1BD3B8K1ANR" H 6950 4334 50  0000 C CNN
 F 2 "Connector_RJ:RJ45_Amphenol_RJMG1BD3B8K1ANR" H 6950 4400 50  0001 C CNN
@@
 U 1 1 5DA5AAEB
 P 6000 4350
-F 0 "#PWR?" H 6000 4100 50  0001 C CNN
+AR Path="/5DA5AAEB" Ref="#PWR?"  Part="1"
+AR Path="/5DA5A719/5DA5AAEB" Ref="#PWR0709"  Part="1"
+F 0 "#PWR0709" H 6000 4100 50  0001 C CNN
 F 1 "GND" H 6005 4177 50  0000 C CNN
 F 2 "" H 6000 4350 50  0001 C CNN
