File: PCB/HeManTCN/Memoria Externa.sch (KiCad schematic (older format))
At the start: 10 parts

Commit message: Hoja A1
Desarme las hojas jerarquicas y configure la hoja del esquematico como A1. Hay lugar suficiente (por ahora) para todo.
Parts:
- gave numbers to parts that had none: 10
Changed lines of the file:
@@
 U 1 1 5DA41C4D
 P 3800 3250
-F 0 "C?" H 3550 3300 50  0000 L CNN
+AR Path="/5DA41C4D" Ref="C?"  Part="1"
+AR Path="/5DA4186F/5DA41C4D" Ref="C401"  Part="1"
+F 0 "C401" H 3550 3300 50  0000 L CNN
 F 1 "0.1u" H 3500 3200 50  0000 L CNN
 F 2 "Capacitor_SMD:C_0805_2012Metric" H 3800 3250 50  0001 C CNN
@@
 U 1 1 5DA41C54
 P 3800 3150
-F 0 "#PWR?" H 3800 3000 50  0001 C CNN
+AR Path="/5DA41C54" Ref="#PWR?"  Part="1"
+AR Path="/5DA4186F/5DA41C54" Ref="#PWR0401"  Part="1"
+F 0 "#PWR0401" H 3800 3000 50  0001 C CNN
 F 1 "+3.3V" H 3815 3323 50  0000 C CNN
 F 2 "" H 3800 3150 50  0001 C CNN
@@
 U 1 1 5DA41C5B
 P 3800 3350
-F 0 "#PWR?" H 3800 3100 50  0001 C CNN
+AR Path="/5DA41C5B" Ref="#PWR?"  Part="1"
+AR Path="/5DA4186F/5DA41C5B" Ref="#PWR0402"  Part="1"
+F 0 "#PWR0402" H 3800 3100 50  0001 C CNN
 F 1 "GND" H 3850 3200 50  0000 R CNN
 F 2 "" H 3800 3350 50  0001 C CNN
@@
 U 1 1 5DA41C62
 P 6850 3750
-F 0 "#PWR?" H 6850 3500 50  0001 C CNN
+AR Path="/5DA41C62" Ref="#PWR?"  Part="1"
+AR Path="/5DA4186F/5DA41C62" Ref="#PWR0406"  Part="1"
+F 0 "#PWR0406" H 6850 3500 50  0001 C CNN
 F 1 "GND" H 6900 3600 50  0000 R CNN
 F 2 "" H 6850 3750 50  0001 C CNN
@@
 U 1 1 5DA41C69
 P 6500 4400
-F 0 "C?" H 6592 4446 50  0000 L CNN
+AR Path="/5DA41C69" Ref="C?"  Part="1"
+AR Path="/5DA4186F/5DA41C69" Ref="C402"  Part="1"
+F 0 "C402" H 6592 4446 50  0000 L CNN
 F 1 "0.1u" H 6592 4355 50  0000 L CNN
 F 2 "Capacitor_SMD:C_0805_2012Metric" H 6500 4400 50  0001 C CNN
@@
 U 1 1 5DA41C70
 P 6500 4300
-F 0 "#PWR?" H 6500 4150 50  0001 C CNN
+AR Path="/5DA41C70" Ref="#PWR?"  Part="1"
+AR Path="/5DA4186F/5DA41C70" Ref="#PWR0404"  Part="1"
+F 0 "#PWR0404" H 6500 4150 50  0001 C CNN
 F 1 "+3.3V" H 6515 4473 50  0000 C CNN
 F 2 "" H 6500 4300 50  0001 C CNN
@@
 U 1 1 5DA41C76
 P 6500 4500
-F 0 "#PWR?" H 6500 4250 50  0001 C CNN
+AR Path="/5DA41C76" Ref="#PWR?"  Part="1"
+AR Path="/5DA4186F/5DA41C76" Ref="#PWR0405"  Part="1"
+F 0 "#PWR0405" H 6500 4250 50  0001 C CNN
 F 1 "GND" H 6505 4327 50  0000 C CNN
 F 2 "" H 6500 4500 50  0001 C CNN
@@
 U 1 1 5DA41C7C
 P 4950 4600
-F 0 "#PWR?" H 4950 4350 50  0001 C CNN
+AR Path="/5DA41C7C" Ref="#PWR?"  Part="1"
+AR Path="/5DA4186F/5DA41C7C" Ref="#PWR0403"  Part="1"
+F 0 "#PWR0403" H 4950 4350 50  0001 C CNN
 F 1 "GND" V 4950 4450 50  0000 R CNN
 F 2 "" H 4950 4600 50  0001 C CNN
@@
 U 1 1 5DA41C8A
 P 3950 4300
-F 0 "U?" H 5475 4587 60  0000 C CNN
+AR Path="/5DA41C8A" Ref="U?"  Part="1"
+AR Path="/5DA4186F/5DA41C8A" Ref="U401"  Part="1"
+F 0 "U401" H 5475 4587 60  0000 C CNN
 F 1 "S25FL127SABMFI101" H 5475 4481 60  0000 C CNN
 F 2 "footprints:S25FL127SABMFI101" H 5450 4540 60  0001 C CNN
@@
 U 1 1 5DA41C95
 P 4450 2850
-F 0 "R?" V 4500 2750 50  0000 R CNN
+AR Path="/5DA41C95" Ref="R?"  Part="1"
+AR Path="/5DA4186F/5DA41C95" Ref="R401"  Part="1"
+F 0 "R401" V 4500 2750 50  0000 R CNN
 F 1 "4K7" V 4500 3100 50  0000 R CNN
 F 2 "Resistor_SMD:R_0805_2012Metric" H 4450 2850 50  0001 C CNN
@@
 U 1 1 5DA41C9F
 P 4450 2950
-F 0 "R?" V 4500 2850 50  0000 R CNN
+AR Path="/5DA41C9F" Ref="R?"  Part="1"
+AR Path="/5DA4186F/5DA41C9F" Ref="R402"  Part="1"
+F 0 "R402" V 4500 2850 50  0000 R CNN
 F 1 "4K7" V 4500 3200 50  0000 R CNN
 F 2 "Resistor_SMD:R_0805_2012Metric" H 4450 2950 50  0001 C CNN
@@
 U 1 1 5DA41CA7
 P 4450 3050
-F 0 "R?" V 4500 2950 50  0000 R CNN
+AR Path="/5DA41CA7" Ref="R?"  Part="1"
+AR Path="/5DA4186F/5DA41CA7" Ref="R403"  Part="1"
+F 0 "R403" V 4500 2950 50  0000 R CNN
 F 1 "4K7" V 4500 3300 50  0000 R CNN
 F 2 "Resistor_SMD:R_0805_2012Metric" H 4450 3050 50  0001 C CNN
@@
 U 1 1 5DA41CAF
 P 4450 3250
-F 0 "R?" V 4500 3150 50  0000 R CNN
+AR Path="/5DA41CAF" Ref="R?"  Part="1"
+AR Path="/5DA4186F/5DA41CAF" Ref="R404"  Part="1"
+F 0 "R404" V 4500 3150 50  0000 R CNN
 F 1 "4K7" V 4500 3500 50  0000 R CNN
 F 2 "Resistor_SMD:R_0805_2012Metric" H 4450 3250 50  0001 C CNN
@@
 U 1 1 5DA41CB7
 P 4450 3450
-F 0 "R?" V 4500 3350 50  0000 R CNN
+AR Path="/5DA41CB7" Ref="R?"  Part="1"
+AR Path="/5DA4186F/5DA41CB7" Ref="R405"  Part="1"
+F 0 "R405" V 4500 3350 50  0000 R CNN
 F 1 "4K7" V 4500 3700 50  0000 R CNN
 F 2 "Resistor_SMD:R_0805_2012Metric" H 4450 3450 50  0001 C CNN
@@
 U 1 1 5DA41CBF
 P 4450 3550
-F 0 "R?" V 4500 3450 50  0000 R CNN
+AR Path="/5DA41CBF" Ref="R?"  Part="1"
+AR Path="/5DA4186F/5DA41CBF" Ref="R406"  Part="1"
+F 0 "R406" V 4500 3450 50  0000 R CNN
 F 1 "4K7" V 4500 3800 50  0000 R CNN
 F 2 "Resistor_SMD:R_0805_2012Metric" H 4450 3550 50  0001 C CNN
@@
 U 1 1 5DA41CC6
 P 6050 3150
-F 0 "J?" H 5350 3750 50  0000 C CNN
+AR Path="/5DA41CC6" Ref="J?"  Part="1"
+AR Path="/5DA4186F/5DA41CC6" Ref="J401"  Part="1"
+F 0 "J401" H 5350 3750 50  0000 C CNN
 F 1 "Micro_SD_Card" H 6000 3750 50  0000 C CNN
 F 2 "Connector_Card:microSD_HC_Hirose_DM3D-SF" H 7200 3450 50  0001 C CNN
