File: PCB/HeManTCN/Protoboard.sch (KiCad schematic (older format))
At the start: 9 parts

Commit message: Hoja A1
Desarme las hojas jerarquicas y configure la hoja del esquematico como A1. Hay lugar suficiente (por ahora) para todo.
Parts:
- gave numbers to parts that had none: 9
Changed lines of the file:
@@
 $Descr A4 11693 8268
 encoding utf-8
-Sheet 6 11
+Sheet 6 3
 Title "SnifferTCN"
 Date "2019-09-25"
@@
 U 1 1 5DA5383B
 P 5450 3000
-F 0 "H?" V 5404 3149 50  0000 L CNN
+AR Path="/5DA5383B" Ref="H?"  Part="1"
+AR Path="/5DA532BE/5DA5383B" Ref="H603"  Part="1"
+F 0 "H603" V 5404 3149 50  0000 L CNN
 F 1 "MountingHole" V 5495 3149 50  0000 L CNN
 F 2 "MountingHole:MountingHole_3.2mm_M3_Pad_Via" H 5450 3000 50  0001 C CNN
@@
 U 1 1 5DA53842
 P 5450 3200
-F 0 "H?" V 5404 3349 50  0000 L CNN
+AR Path="/5DA53842" Ref="H?"  Part="1"
+AR Path="/5DA532BE/5DA53842" Ref="H604"  Part="1"
+F 0 "H604" V 5404 3349 50  0000 L CNN
 F 1 "MountingHole" V 5495 3349 50  0000 L CNN
 F 2 "MountingHole:MountingHole_3.2mm_M3_Pad_Via" H 5450 3200 50  0001 C CNN
@@
 U 1 1 5DA53849
 P 5250 3000
-F 0 "H?" V 5200 3200 50  0000 C CNN
+AR Path="/5DA53849" Ref="H?"  Part="1"
+AR Path="/5DA532BE/5DA53849" Ref="H601"  Part="1"
+F 0 "H601" V 5200 3200 50  0000 C CNN
 F 1 "MountingHole" V 5300 3400 50  0000 C CNN
 F 2 "MountingHole:MountingHole_3.2mm_M3_Pad_Via" H 5250 3000 50  0001 C CNN
@@
 U 1 1 5DA53850
 P 5250 3200
-F 0 "H?" V 5204 3350 50  0000 L CNN
+AR Path="/5DA53850" Ref="H?"  Part="1"
+AR Path="/5DA532BE/5DA53850" Ref="H602"  Part="1"
+F 0 "H602" V 5204 3350 50  0000 L CNN
 F 1 "MountingHole" V 5295 3350 50  0000 L CNN
 F 2 "MountingHole:MountingHole_3.2mm_M3_Pad_Via" H 5250 3200 50  0001 C CNN
@@
 U 1 1 5DA5385A
 P 5350 3200
-F 0 "#PWR?" H 5350 2950 50  0001 C CNN
+AR Path="/5DA5385A" Ref="#PWR?"  Part="1"
+AR Path="/5DA532BE/5DA5385A" Ref="#PWR0606"  Part="1"
+F 0 "#PWR0606" H 5350 2950 50  0001 C CNN
 F 1 "GND" H 5355 3027 50  0000 C CNN
 F 2 "" H 5350 3200 50  0001 C CNN
@@
 U 1 1 5DA53874
 P 3950 3850
-F 0 "#PWR?" H 3950 3600 50  0001 C CNN
+AR Path="/5DA53874" Ref="#PWR?"  Part="1"
+AR Path="/5DA532BE/5DA53874" Ref="#PWR0601"  Part="1"
+F 0 "#PWR0601" H 3950 3600 50  0001 C CNN
 F 1 "GND" V 3950 3700 50  0000 R CNN
 F 2 "" H 3950 3850 50  0001 C CNN
@@
 U 1 1 5DA5387A
 P 4450 3850
-F 0 "#PWR?" H 4450 3700 50  0001 C CNN
+AR Path="/5DA5387A" Ref="#PWR?"  Part="1"
+AR Path="/5DA532BE/5DA5387A" Ref="#PWR0604"  Part="1"
+F 0 "#PWR0604" H 4450 3700 50  0001 C CNN
 F 1 "+3.3V" V 4465 3978 50  0000 L CNN
 F 2 "" H 4450 3850 50  0001 C CNN
@@
 U 1 1 5DA53893
 P 6100 3850
-F 0 "#PWR?" H 6100 3700 50  0001 C CNN
+AR Path="/5DA53893" Ref="#PWR?"  Part="1"
+AR Path="/5DA532BE/5DA53893" Ref="#PWR0610"  Part="1"
+F 0 "#PWR0610" H 6100 3700 50  0001 C CNN
 F 1 "+3.3V" V 6115 3978 50  0000 L CNN
 F 2 "" H 6100 3850 50  0001 C CNN
@@
 U 1 1 5DA53899
 P 6600 3750
-F 0 "#PWR?" H 6600 3500 50  0001 C CNN
+AR Path="/5DA53899" Ref="#PWR?"  Part="1"
+AR Path="/5DA532BE/5DA53899" Ref="#PWR0611"  Part="1"
+F 0 "#PWR0611" H 6600 3500 50  0001 C CNN
 F 1 "GND" V 6605 3622 50  0000 R CNN
 F 2 "" H 6600 3750 50  0001 C CNN
@@
 U 1 1 5DA538AB
 P 4900 4950
-F 0 "#PWR?" H 4900 4700 50  0001 C CNN
+AR Path="/5DA538AB" Ref="#PWR?"  Part="1"
+AR Path="/5DA532BE/5DA538AB" Ref="#PWR0605"  Part="1"
+F 0 "#PWR0605" H 4900 4700 50  0001 C CNN
 F 1 "GND" V 4905 4822 50  0000 R CNN
 F 2 "" H 4900 4950 50  0001 C CNN
@@
 U 1 1 5DA538C1
 P 4350 2150
-F 0 "#PWR?" H 4350 1900 50  0001 C CNN
+AR Path="/5DA538C1" Ref="#PWR?"  Part="1"
+AR Path="/5DA532BE/5DA538C1" Ref="#PWR0602"  Part="1"
+F 0 "#PWR0602" H 4350 1900 50  0001 C CNN
 F 1 "GND" V 4355 2022 50  0000 R CNN
 F 2 "" H 4350 2150 50  0001 C CNN
@@
 U 1 1 5DA538C7
 P 5500 2650
-F 0 "#PWR?" H 5500 2400 50  0001 C CNN
+AR Path="/5DA538C7" Ref="#PWR?"  Part="1"
+AR Path="/5DA532BE/5DA538C7" Ref="#PWR0608"  Part="1"
+F 0 "#PWR0608" H 5500 2400 50  0001 C CNN
 F 1 "GND" V 5505 2522 50  0000 R CNN
 F 2 "" H 5500 2650 50  0001 C CNN
@@
 U 1 1 5DA538CD
 P 5500 2150
-F 0 "#PWR?" H 5500 2000 50  0001 C CNN
+AR Path="/5DA538CD" Ref="#PWR?"  Part="1"
+AR Path="/5DA532BE/5DA538CD" Ref="#PWR0607"  Part="1"
+F 0 "#PWR0607" H 5500 2000 50  0001 C CNN
 F 1 "+3.3V" V 5515 2278 50  0000 L CNN
 F 2 "" H 5500 2150 50  0001 C CNN
@@
 U 1 1 5DA538D4
 P 4350 2650
-F 0 "#PWR?" H 4350 2550 50  0001 C CNN
+AR Path="/5DA538D4" Ref="#PWR?"  Part="1"
+AR Path="/5DA532BE/5DA538D4" Ref="#PWR0603"  Part="1"
+F 0 "#PWR0603" H 4350 2550 50  0001 C CNN
 F 1 "VDC" H 4350 2950 50  0000 C CNN
 F 2 "" H 4350 2650 50  0001 C CNN
@@
 U 1 1 5DA538E9
 P 4150 4350
-F 0 "J?" H 4200 3525 50  0000 C CNN
+AR Path="/5DA538E9" Ref="J?"  Part="1"
+AR Path="/5DA532BE/5DA538E9" Ref="J602"  Part="1"
+F 0 "J602" H 4200 3525 50  0000 C CNN
 F 1 "Conn_02x12_Odd_Even" H 4200 3616 50  0000 C CNN
 F 2 "Connector_PinSocket_2.54mm:PinSocket_2x12_P2.54mm_Vertical" H 4150 4350 50  0001 C CNN
@@
 U 1 1 5DA538F3
 P 5400 4250
-F 0 "J?" H 5450 4967 50  0000 C CNN
+AR Path="/5DA538F3" Ref="J?"  Part="1"
+AR Path="/5DA532BE/5DA538F3" Ref="J603"  Part="1"
+F 0 "J603" H 5450 4967 50  0000 C CNN
 F 1 "Conn_02x12_Odd_Even" H 5450 4876 50  0000 C CNN
 F 2 "Connector_PinSocket_2.54mm:PinSocket_2x12_P2.54mm_Vertical" H 5400 4250 50  0001 C CNN
@@
 U 1 1 5DA53914
 P 6400 4250
-F 0 "J?" H 6450 4967 50  0000 C CNN
+AR Path="/5DA53914" Ref="J?"  Part="1"
+AR Path="/5DA532BE/5DA53914" Ref="J605"  Part="1"
+F 0 "J605" H 6450 4967 50  0000 C CNN
 F 1 "Conn_02x12_Odd_Even" H 6450 4876 50  0000 C CNN
 F 2 "Connector_PinSocket_2.54mm:PinSocket_2x12_P2.54mm_Vertical" H 6400 4250 50  0001 C CNN
@@
 U 1 1 5DA5391C
 P 6900 3850
-F 0 "#PWR?" H 6900 3700 50  0001 C CNN
+AR Path="/5DA5391C" Ref="#PWR?"  Part="1"
+AR Path="/5DA532BE/5DA5391C" Ref="#PWR0612"  Part="1"
+F 0 "#PWR0612" H 6900 3700 50  0001 C CNN
 F 1 "+BATT" V 6915 3978 50  0000 L CNN
 F 2 "" H 6900 3850 50  0001 C CNN
@@
 U 1 1 5DA53923
 P 5850 2350
-F 0 "J?" V 5854 2630 50  0000 L CNN
+AR Path="/5DA53923" Ref="J?"  Part="1"
+AR Path="/5DA532BE/5DA53923" Ref="J604"  Part="1"
+F 0 "J604" V 5854 2630 50  0000 L CNN
 F 1 "Conn_02x05_Odd_Even" V 5945 2630 50  0000 L CNN
 F 2 "Connector_PinSocket_2.54mm:PinSocket_2x05_P2.54mm_Vertical" H 5850 2350 50  0001 C CNN
@@
 U 1 1 5DA5392A
 P 4150 2350
-F 0 "J?" V 4154 2630 50  0000 L CNN
+AR Path="/5DA5392A" Ref="J?"  Part="1"
+AR Path="/5DA532BE/5DA5392A" Ref="J601"  Part="1"
+F 0 "J601" V 4154 2630 50  0000 L CNN
 F 1 "Conn_02x05_Odd_Even" V 4245 2630 50  0000 L CNN
 F 2 "Connector_PinSocket_2.54mm:PinSocket_2x05_P2.54mm_Vertical" H 4150 2350 50  0001 C CNN
@@
 U 1 1 5DA53937
 P 6100 3750
-F 0 "#PWR?" H 6100 3500 50  0001 C CNN
+AR Path="/5DA53937" Ref="#PWR?"  Part="1"
+AR Path="/5DA532BE/5DA53937" Ref="#PWR0609"  Part="1"
+F 0 "#PWR0609" H 6100 3500 50  0001 C CNN
 F 1 "GND" V 6105 3622 50  0000 R CNN
 F 2 "" H 6100 3750 50  0001 C CNN
