File: PCB/HeManTCN/RS485.sch (KiCad schematic (older format))
At the start: 13 parts

Commit message: Hoja A1
Desarme las hojas jerarquicas y configure la hoja del esquematico como A1. Hay lugar suficiente (por ahora) para todo.
Parts:
- gave numbers to parts that had none: 13
Changed lines of the file:
@@
 $Descr A4 11693 8268
 encoding utf-8
-Sheet 10 11
+Sheet 10 8
 Title "SnifferTCN"
 Date "2019-09-25"
@@
 U 1 1 5DA5FCAD
 P 4625 4625
-F 0 "U?" H 4625 5203 50  0000 C CNN
+AR Path="/5DA5FCAD" Ref="U?"  Part="1"
+AR Path="/5DA5FACD/5DA5FCAD" Ref="U1002"  Part="1"
+F 0 "U1002" H 4625 5203 50  0000 C CNN
 F 1 "ISL83483" H 4625 5112 50  0000 C CNN
 F 2 "Package_SO:SOIC-8_3.9x4.9mm_P1.27mm" H 4625 3725 50  0001 C CNN
@@
 	1    0    0    -1
 $EndComp
-Text Label 4225 4825 2    50   ~ 0
-RS485_TX
-Text Label 4225 4525 2    50   ~ 0
-RS485_RX
 Text Label 4225 4625 2    50   ~ 0
 RS485_DE
@@
 U 1 1 5DA5FCBB
 P 6750 4350
-F 0 "J?" H 6750 4650 50  0000 C CNN
+AR Path="/5DA5FCBB" Ref="J?"  Part="1"
+AR Path="/5DA5FACD/5DA5FCBB" Ref="J1001"  Part="1"
+F 0 "J1001" H 6750 4650 50  0000 C CNN
 F 1 "Screw_Terminal_01x06" V 6850 4350 50  0000 C CNN
 F 2 "Connectors_Phoenix:PhoenixContact_MC-G_06x5.08mm_Angled" H 6750 4350 50  0001 C CNN
@@
 U 1 1 5DA5FCC7
 P 5900 4550
-F 0 "D?" V 5558 4550 50  0000 C CNN
+AR Path="/5DA5FCC7" Ref="D?"  Part="1"
+AR Path="/5DA5FACD/5DA5FCC7" Ref="D1002"  Part="1"
+F 0 "D1002" V 5558 4550 50  0000 C CNN
 F 1 "NUP2105L" V 5649 4550 50  0000 C CNN
 F 2 "Package_TO_SOT_SMD:SOT-23" H 6125 4500 50  0001 L CNN
@@
 U 1 1 5DA5FCCF
 P 5900 4200
-F 0 "D?" V 6242 4200 50  0000 C CNN
+AR Path="/5DA5FCCF" Ref="D?"  Part="1"
+AR Path="/5DA5FACD/5DA5FCCF" Ref="D1001"  Part="1"
+F 0 "D1001" V 6242 4200 50  0000 C CNN
 F 1 "NUP2105L" V 6151 4200 50  0000 C CNN
 F 2 "Package_TO_SOT_SMD:SOT-23" H 6125 4150 50  0001 L CNN
@@
 U 1 1 5DA5FCE6
 P 4575 3000
-F 0 "#PWR?" H 4575 2850 50  0001 C CNN
+AR Path="/5DA5FCE6" Ref="#PWR?"  Part="1"
+AR Path="/5DA5FACD/5DA5FCE6" Ref="#PWR01001"  Part="1"
+F 0 "#PWR01001" H 4575 2850 50  0001 C CNN
 F 1 "+3.3V" V 4590 3128 50  0000 L CNN
 F 2 "" H 4575 3000 50  0001 C CNN
@@
 U 1 1 5DA5FCF0
 P 5150 4225
-F 0 "#PWR?" H 5150 3975 50  0001 C CNN
+AR Path="/5DA5FCF0" Ref="#PWR?"  Part="1"
+AR Path="/5DA5FACD/5DA5FCF0" Ref="#PWR01008"  Part="1"
+F 0 "#PWR01008" H 5150 3975 50  0001 C CNN
 F 1 "GND" V 5155 4097 50  0000 R CNN
 F 2 "" H 5150 4225 50  0001 C CNN
@@
 U 1 1 5DA5FCF7
 P 4575 3400
-F 0 "U?" H 4575 3978 50  0000 C CNN
+AR Path="/5DA5FCF7" Ref="U?"  Part="1"
+AR Path="/5DA5FACD/5DA5FCF7" Ref="U1001"  Part="1"
+F 0 "U1001" H 4575 3978 50  0000 C CNN
 F 1 "TCAN332" H 4575 3887 50  0000 C CNN
 F 2 "Package_TO_SOT_SMD:SOT-23-8" H 4575 2900 50  0001 C CIN
@@
 U 1 1 5DA5FCFF
 P 6375 2825
-F 0 "R?" V 6300 2825 50  0000 C CNN
+AR Path="/5DA5FCFF" Ref="R?"  Part="1"
+AR Path="/5DA5FACD/5DA5FCFF" Ref="R1003"  Part="1"
+F 0 "R1003" V 6300 2825 50  0000 C CNN
 F 1 "2K2" V 6450 2825 50  0000 C CNN
 F 2 "Resistor_SMD:R_0805_2012Metric" H 6375 2825 50  0001 C CNN
@@
 U 1 1 5DA5FD07
 P 6375 3025
-F 0 "R?" V 6300 3025 50  0000 C CNN
+AR Path="/5DA5FD07" Ref="R?"  Part="1"
+AR Path="/5DA5FACD/5DA5FD07" Ref="R1004"  Part="1"
+F 0 "R1004" V 6300 3025 50  0000 C CNN
 F 1 "120R" V 6450 3025 50  0000 C CNN
 F 2 "Resistor_SMD:R_0805_2012Metric" H 6375 3025 50  0001 C CNN
@@
 U 1 1 5DA5FD0F
 P 6375 3225
-F 0 "R?" V 6300 3225 50  0000 C CNN
+AR Path="/5DA5FD0F" Ref="R?"  Part="1"
+AR Path="/5DA5FACD/5DA5FD0F" Ref="R1005"  Part="1"
+F 0 "R1005" V 6300 3225 50  0000 C CNN
 F 1 "2K2" V 6450 3225 50  0000 C CNN
 F 2 "Resistor_SMD:R_0805_2012Metric" H 6375 3225 50  0001 C CNN
@@
 U 1 1 5DA5FD1D
 P 5800 3025
-F 0 "R?" H 5858 2979 50  0000 L CNN
+AR Path="/5DA5FD1D" Ref="R?"  Part="1"
+AR Path="/5DA5FACD/5DA5FD1D" Ref="R1001"  Part="1"
+F 0 "R1001" H 5858 2979 50  0000 L CNN
 F 1 "60R" H 5858 3070 50  0000 L CNN
 F 2 "Resistor_SMD:R_0805_2012Metric" H 5800 3025 50  0001 C CNN
@@
 U 1 1 5DA5FD25
 P 6025 3025
-F 0 "R?" H 5966 2979 50  0000 R CNN
+AR Path="/5DA5FD25" Ref="R?"  Part="1"
+AR Path="/5DA5FACD/5DA5FD25" Ref="R1002"  Part="1"
+F 0 "R1002" H 5966 2979 50  0000 R CNN
 F 1 "60R" H 5966 3070 50  0000 R CNN
 F 2 "Resistor_SMD:R_0805_2012Metric" H 6025 3025 50  0001 C CNN
@@
 U 1 1 5DA5FD2D
 P 5900 3225
-F 0 "C?" H 5992 3271 50  0000 L CNN
+AR Path="/5DA5FD2D" Ref="C?"  Part="1"
+AR Path="/5DA5FACD/5DA5FD2D" Ref="C1003"  Part="1"
+F 0 "C1003" H 5992 3271 50  0000 L CNN
 F 1 "10p" H 5992 3180 50  0000 L CNN
 F 2 "Capacitor_SMD:C_0805_2012Metric" H 5900 3225 50  0001 C CNN
@@
 U 1 1 5DA5FD39
 P 4625 5125
-F 0 "#PWR?" H 4625 4875 50  0001 C CNN
+AR Path="/5DA5FD39" Ref="#PWR?"  Part="1"
+AR Path="/5DA5FACD/5DA5FD39" Ref="#PWR01004"  Part="1"
+F 0 "#PWR01004" H 4625 4875 50  0001 C CNN
 F 1 "GND" V 4630 4997 50  0000 R CNN
 F 2 "" H 4625 5125 50  0001 C CNN
@@
 U 1 1 5DA5FD3F
 P 4625 4225
-F 0 "#PWR?" H 4625 4075 50  0001 C CNN
+AR Path="/5DA5FD3F" Ref="#PWR?"  Part="1"
+AR Path="/5DA5FACD/5DA5FD3F" Ref="#PWR01003"  Part="1"
+F 0 "#PWR01003" H 4625 4075 50  0001 C CNN
 F 1 "+3.3V" V 4640 4353 50  0000 L CNN
 F 2 "" H 4625 4225 50  0001 C CNN
@@
 U 1 1 5DA5FD45
 P 6375 2725
-F 0 "#PWR?" H 6375 2575 50  0001 C CNN
+AR Path="/5DA5FD45" Ref="#PWR?"  Part="1"
+AR Path="/5DA5FACD/5DA5FD45" Ref="#PWR01011"  Part="1"
+F 0 "#PWR01011" H 6375 2575 50  0001 C CNN
 F 1 "+3.3V" H 6390 2898 50  0000 C CNN
 F 2 "" H 6375 2725 50  0001 C CNN
@@
 U 1 1 5DA5FD4B
 P 6150 4950
-F 0 "#PWR?" H 6150 4700 50  0001 C CNN
+AR Path="/5DA5FD4B" Ref="#PWR?"  Part="1"
+AR Path="/5DA5FACD/5DA5FD4B" Ref="#PWR01010"  Part="1"
+F 0 "#PWR01010" H 6150 4700 50  0001 C CNN
 F 1 "GND" V 6155 4822 50  0000 R CNN
 F 2 "" H 6150 4950 50  0001 C CNN
@@
 U 1 1 5DA5FD51
 P 5900 3325
-F 0 "#PWR?" H 5900 3075 50  0001 C CNN
+AR Path="/5DA5FD51" Ref="#PWR?"  Part="1"
+AR Path="/5DA5FACD/5DA5FD51" Ref="#PWR01009"  Part="1"
+F 0 "#PWR01009" H 5900 3075 50  0001 C CNN
 F 1 "GND" H 5905 3152 50  0000 C CNN
 F 2 "" H 5900 3325 50  0001 C CNN
@@
 U 1 1 5DA5FD57
 P 6375 3325
-F 0 "#PWR?" H 6375 3075 50  0001 C CNN
+AR Path="/5DA5FD57" Ref="#PWR?"  Part="1"
+AR Path="/5DA5FACD/5DA5FD57" Ref="#PWR01012"  Part="1"
+F 0 "#PWR01012" H 6375 3075 50  0001 C CNN
 F 1 "GND" H 6380 3152 50  0000 C CNN
 F 2 "" H 6375 3325 50  0001 C CNN
@@
 U 1 1 5DA5FD60
 P 5075 2675
-F 0 "C?" H 5167 2721 50  0000 L CNN
+AR Path="/5DA5FD60" Ref="C?"  Part="1"
+AR Path="/5DA5FACD/5DA5FD60" Ref="C1001"  Part="1"
+F 0 "C1001" H 5167 2721 50  0000 L CNN
 F 1 "0.1u" H 5167 2630 50  0000 L CNN
 F 2 "Capacitor_SMD:C_0805_2012Metric" H 5075 2675 50  0001 C CNN
@@
 U 1 1 5DA5FD68
 P 5150 4125
-F 0 "C?" H 5242 4171 50  0000 L CNN
+AR Path="/5DA5FD68" Ref="C?"  Part="1"
+AR Path="/5DA5FACD/5DA5FD68" Ref="C1002"  Part="1"
+F 0 "C1002" H 5242 4171 50  0000 L CNN
 F 1 "0.1u" H 5242 4080 50  0000 L CNN
 F 2 "Capacitor_SMD:C_0805_2012Metric" H 5150 4125 50  0001 C CNN
@@
 U 1 1 5DA5FD6F
 P 5150 4025
-F 0 "#PWR?" H 5150 3875 50  0001 C CNN
+AR Path="/5DA5FD6F" Ref="#PWR?"  Part="1"
+AR Path="/5DA5FACD/5DA5FD6F" Ref="#PWR01007"  Part="1"
+F 0 "#PWR01007" H 5150 3875 50  0001 C CNN
 F 1 "+3.3V" V 5165 4153 50  0000 L CNN
 F 2 "" H 5150 4025 50  0001 C CNN
@@
 U 1 1 5DA5FD75
 P 4575 3800
-F 0 "#PWR?" H 4575 3550 50  0001 C CNN
+AR Path="/5DA5FD75" Ref="#PWR?"  Part="1"
+AR Path="/5DA5FACD/5DA5FD75" Ref="#PWR01002"  Part="1"
+F 0 "#PWR01002" H 4575 3550 50  0001 C CNN
 F 1 "GND" V 4580 3672 50  0000 R CNN
 F 2 "" H 4575 3800 50  0001 C CNN
@@
 U 1 1 5DA5FD7B
 P 5075 2575
-F 0 "#PWR?" H 5075 2425 50  0001 C CNN
+AR Path="/5DA5FD7B" Ref="#PWR?"  Part="1"
+AR Path="/5DA5FACD/5DA5FD7B" Ref="#PWR01005"  Part="1"
+F 0 "#PWR01005" H 5075 2425 50  0001 C CNN
 F 1 "+3.3V" V 5090 2703 50  0000 L CNN
 F 2 "" H 5075 2575 50  0001 C CNN
@@
 U 1 1 5DA5FD81
 P 5075 2775
-F 0 "#PWR?" H 5075 2525 50  0001 C CNN
+AR Path="/5DA5FD81" Ref="#PWR?"  Part="1"
+AR Path="/5DA5FACD/5DA5FD81" Ref="#PWR01006"  Part="1"
+F 0 "#PWR01006" H 5075 2525 50  0001 C CNN
 F 1 "GND" V 5080 2647 50  0000 R CNN
 F 2 "" H 5075 2775 50  0001 C CNN
@@
 	0    1    1    0
 $EndComp
+Text GLabel 4225 4525 0    50   Input ~ 0
+RS485_RX
+Text GLabel 4225 4825 0    50   Input ~ 0
+RS485_TX
 $EndSCHEMATC
