File: PCB/HeManTCN/USB.sch (KiCad schematic (older format))
At the start: 9 parts

Commit message: Hoja A1
Desarme las hojas jerarquicas y configure la hoja del esquematico como A1. Hay lugar suficiente (por ahora) para todo.
Parts:
- gave numbers to parts that had none: 9
Changed lines of the file:
@@
 $Descr A4 11693 8268
 encoding utf-8
-Sheet 5 11
+Sheet 5 8
 Title "SnifferTCN"
 Date "2019-09-25"
@@
 U 1 1 5DA4DEF7
 P 6550 2500
-F 0 "#PWR?" H 6550 2250 50  0001 C CNN
+AR Path="/5DA4DEF7" Ref="#PWR?"  Part="1"
+AR Path="/5DA4DC5D/5DA4DEF7" Ref="#PWR0506"  Part="1"
+F 0 "#PWR0506" H 6550 2250 50  0001 C CNN
 F 1 "GND" V 6555 2372 50  0000 R CNN
 F 2 "" H 6550 2500 50  0001 C CNN
@@
 U 1 1 5DA4DEFD
 P 6550 3400
-F 0 "#PWR?" H 6550 3150 50  0001 C CNN
+AR Path="/5DA4DEFD" Ref="#PWR?"  Part="1"
+AR Path="/5DA4DC5D/5DA4DEFD" Ref="#PWR0507"  Part="1"
+F 0 "#PWR0507" H 6550 3150 50  0001 C CNN
 F 1 "GND" V 6555 3272 50  0000 R CNN
 F 2 "" H 6550 3400 50  0001 C CNN
@@
 U 1 1 5DA4DF05
 P 4900 3000
-F 0 "#PWR?" H 4900 2750 50  0001 C CNN
+AR Path="/5DA4DF05" Ref="#PWR?"  Part="1"
+AR Path="/5DA4DC5D/5DA4DF05" Ref="#PWR0502"  Part="1"
+F 0 "#PWR0502" H 4900 2750 50  0001 C CNN
 F 1 "GND" V 4905 2872 50  0000 R CNN
 F 2 "" H 4900 3000 50  0001 C CNN
@@
 U 1 1 5DA4DF12
 P 4900 4250
-F 0 "#PWR?" H 4900 4000 50  0001 C CNN
+AR Path="/5DA4DF12" Ref="#PWR?"  Part="1"
+AR Path="/5DA4DC5D/5DA4DF12" Ref="#PWR0503"  Part="1"
+F 0 "#PWR0503" H 4900 4000 50  0001 C CNN
 F 1 "GND" V 4905 4122 50  0000 R CNN
 F 2 "" H 4900 4250 50  0001 C CNN
@@
 U 1 1 5DA4DF19
 P 4850 5450
-F 0 "#PWR?" H 4850 5200 50  0001 C CNN
+AR Path="/5DA4DF19" Ref="#PWR?"  Part="1"
+AR Path="/5DA4DC5D/5DA4DF19" Ref="#PWR0501"  Part="1"
+F 0 "#PWR0501" H 4850 5200 50  0001 C CNN
 F 1 "GND" V 4855 5322 50  0000 R CNN
 F 2 "" H 4850 5450 50  0001 C CNN
@@
 U 1 1 5DA4DF28
 P 4900 2500
-F 0 "U?" H 4650 2850 50  0000 C CNN
+AR Path="/5DA4DF28" Ref="U?"  Part="1"
+AR Path="/5DA4DC5D/5DA4DF28" Ref="U502"  Part="1"
+F 0 "U502" H 4650 2850 50  0000 C CNN
 F 1 "USBLC6-2SC6" H 5250 2850 50  0000 C CNN
 F 2 "Package_TO_SOT_SMD:SOT-23-6" H 4150 2900 50  0001 C CNN
@@
 U 1 1 5DA4DF30
 P 4900 3750
-F 0 "U?" H 4650 4100 50  0000 C CNN
+AR Path="/5DA4DF30" Ref="U?"  Part="1"
+AR Path="/5DA4DC5D/5DA4DF30" Ref="U503"  Part="1"
+F 0 "U503" H 4650 4100 50  0000 C CNN
 F 1 "USBLC6-2SC6" H 5250 4100 50  0000 C CNN
 F 2 "Package_TO_SOT_SMD:SOT-23-6" H 4150 4150 50  0001 C CNN
@@
 U 1 1 5DA4DF38
 P 4850 4950
-F 0 "U?" H 4600 5300 50  0000 C CNN
+AR Path="/5DA4DF38" Ref="U?"  Part="1"
+AR Path="/5DA4DC5D/5DA4DF38" Ref="U501"  Part="1"
+F 0 "U501" H 4600 5300 50  0000 C CNN
 F 1 "USBLC6-2SC6" H 5250 5300 50  0000 C CNN
 F 2 "Package_TO_SOT_SMD:SOT-23-6" H 4100 5350 50  0001 C CNN
@@
 U 1 1 5DA4DF43
 P 6550 2100
-F 0 "J?" H 6750 2450 50  0000 R CNN
+AR Path="/5DA4DF43" Ref="J?"  Part="1"
+AR Path="/5DA4DC5D/5DA4DF43" Ref="J501"  Part="1"
+F 0 "J501" H 6750 2450 50  0000 R CNN
 F 1 "USB_B" H 6600 2450 50  0000 R CNN
 F 2 "Connector_USB:USB_B_OST_USB-B1HSxx_Horizontal" H 6700 2050 50  0001 C CNN
@@
 U 1 1 5DA4DF4D
 P 6550 3000
-F 0 "J?" H 6750 3350 50  0000 R CNN
+AR Path="/5DA4DF4D" Ref="J?"  Part="1"
+AR Path="/5DA4DC5D/5DA4DF4D" Ref="J502"  Part="1"
+F 0 "J502" H 6750 3350 50  0000 R CNN
 F 1 "USB_B" H 6600 3350 50  0000 R CNN
 F 2 "Connector_USB:USB_B_OST_USB-B1HSxx_Horizontal" H 6700 2950 50  0001 C CNN
@@
 U 1 1 5DA4DF56
 P 5900 4200
-F 0 "#PWR?" H 5900 4100 50  0001 C CNN
+AR Path="/5DA4DF56" Ref="#PWR?"  Part="1"
+AR Path="/5DA4DC5D/5DA4DF56" Ref="#PWR0505"  Part="1"
+F 0 "#PWR0505" H 5900 4100 50  0001 C CNN
 F 1 "VDC" H 5900 4475 50  0000 C CNN
 F 2 "" H 5900 4200 50  0001 C CNN
@@
 U 1 1 5DA4DF5D
 P 6350 4400
-F 0 "U?" H 6350 4765 50  0000 C CNN
+AR Path="/5DA4DF5D" Ref="U?"  Part="1"
+AR Path="/5DA4DC5D/5DA4DF5D" Ref="U504"  Part="1"
+F 0 "U504" H 6350 4765 50  0000 C CNN
 F 1 "MIC2005A" H 6350 4674 50  0000 C CNN
 F 2 "Package_TO_SOT_SMD:SOT-23-5" H 6350 4400 50  0001 C CNN
@@
 U 1 1 5DA4DF6B
 P 7100 4400
-F 0 "C?" H 7192 4446 50  0000 L CNN
+AR Path="/5DA4DF6B" Ref="C?"  Part="1"
+AR Path="/5DA4DC5D/5DA4DF6B" Ref="C502"  Part="1"
+F 0 "C502" H 7192 4446 50  0000 L CNN
 F 1 "2.2u" H 7192 4355 50  0000 L CNN
 F 2 "Capacitor_SMD:C_0805_2012Metric" H 7100 4400 50  0001 C CNN
@@
 U 1 1 5DA4DF72
 P 7100 4600
-F 0 "#PWR?" H 7100 4350 50  0001 C CNN
+AR Path="/5DA4DF72" Ref="#PWR?"  Part="1"
+AR Path="/5DA4DC5D/5DA4DF72" Ref="#PWR0510"  Part="1"
+F 0 "#PWR0510" H 7100 4350 50  0001 C CNN
 F 1 "GND" V 7105 4472 50  0000 R CNN
 F 2 "" H 7100 4600 50  0001 C CNN
@@
 U 1 1 5DA4DF7B
 P 5700 4300
-F 0 "C?" V 5471 4300 50  0000 C CNN
+AR Path="/5DA4DF7B" Ref="C?"  Part="1"
+AR Path="/5DA4DC5D/5DA4DF7B" Ref="C501"  Part="1"
+F 0 "C501" V 5471 4300 50  0000 C CNN
 F 1 "2.2u" V 5562 4300 50  0000 C CNN
 F 2 "Capacitor_SMD:C_0805_2012Metric" H 5700 4300 50  0001 C CNN
@@
 U 1 1 5DA4DF84
 P 5600 4300
-F 0 "#PWR?" H 5600 4050 50  0001 C CNN
+AR Path="/5DA4DF84" Ref="#PWR?"  Part="1"
+AR Path="/5DA4DC5D/5DA4DF84" Ref="#PWR0504"  Part="1"
+F 0 "#PWR0504" H 5600 4050 50  0001 C CNN
 F 1 "GND" V 5605 4172 50  0000 R CNN
 F 2 "" H 5600 4300 50  0001 C CNN
@@
 U 1 1 5DA4DF94
 P 6850 5150
-F 0 "J?" H 6747 5195 60  0000 R CNN
+AR Path="/5DA4DF94" Ref="J?"  Part="1"
+AR Path="/5DA4DC5D/5DA4DF94" Ref="J503"  Part="1"
+F 0 "J503" H 6747 5195 60  0000 R CNN
 F 1 "73725-0110BLF" H 7550 5550 60  0000 R CNN
 F 2 "footprints:USB_A_Female_Vertical_RA_73725-0110BLF" H 7050 5350 60  0001 L CNN
@@
 U 1 1 5DA4DF9B
 P 6550 4950
-F 0 "#PWR?" H 6550 4700 50  0001 C CNN
+AR Path="/5DA4DF9B" Ref="#PWR?"  Part="1"
+AR Path="/5DA4DC5D/5DA4DF9B" Ref="#PWR0508"  Part="1"
+F 0 "#PWR0508" H 6550 4700 50  0001 C CNN
 F 1 "GND" V 6555 4822 50  0000 R CNN
 F 2 "" H 6550 4950 50  0001 C CNN
@@
 U 1 1 5DA4DFA1
 P 6725 5475
-F 0 "#PWR?" H 6725 5225 50  0001 C CNN
+AR Path="/5DA4DFA1" Ref="#PWR?"  Part="1"
+AR Path="/5DA4DC5D/5DA4DFA1" Ref="#PWR0509"  Part="1"
+F 0 "#PWR0509" H 6725 5225 50  0001 C CNN
 F 1 "GND" V 6730 5347 50  0000 R CNN
 F 2 "" H 6725 5475 50  0001 C CNN
