File: PCB/HeManTCN/HeManTCN.sch (KiCad schematic (older format))
At the start: 108 parts

Commit message: MVBC02D Component 50%
50 % del QFP100 del MVBC02D
Parts:
- added U112: MVBC02D, Package_QFP:LQFP-100_14x14mm_P0.5mm, symbol MCU_ST_STM32H7:STM32H743VITx
- gave numbers to parts that had none: 108
Other:
- note added: "TCN - WTB"
- moved on the sheet: C130, C131, C132, C134, D101, D102, D103, D104, D105, J109, J110, J111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

Commit message: MVBC02D y Sheets
Componente MVBC02D 100%
Hojas jerarquicas listas.
Parts:
- removed C101, C102, C103, C106, C107, C109, C110, C111, C112, C114, C116, C117, C124, C125, C126, C127, C128, C131, C133, C135, C136, C137: 0.1u, Capacitor_SMD:C_0805_2012Metric, symbol Device:C_Small
- removed C104, C105: 18p, Capacitor_SMD:C_0805_2012Metric, symbol Device:C_Small
- removed C108, C121, C123: 4.7u, Capacitor_SMD:C_0805_2012Metric, symbol Device:C_Small
- removed C113, C115, C138: 10p, Capacitor_SMD:C_0805_2012Metric, symbol Device:C_Small
- removed C118, C119: 22p, Capacitor_SMD:C_0805_2012Metric, symbol Device:C_Small
- removed C120, C122, C129, C132, C134: 2.2u, Capacitor_SMD:C_0805_2012Metric, symbol Device:C_Small
- removed C130: 10u, Capacitor_SMD:C_0805_2012Metric, symbol Device:C_Small
- removed D101: LED_PWR, LED_SMD:LED_0805_2012Metric_Castellated, symbol Device:LED_Small_ALT
- removed D102: LED_PC2, LED_SMD:LED_0805_2012Metric_Castellated, symbol Device:LED_Small_ALT
- removed D103, D104, D105: B120-E3, Diode_SMD:D_SOD-123, symbol Diode:B120-E3
- removed D106, D107: NUP2105L, Package_TO_SOT_SMD:SOT-23, symbol Power_Protection:NUP2105L
- removed H101, H102, H103, H104: MountingHole, MountingHole:MountingHole_3.2mm_M3_Pad_Via, symbol Mechanical:MountingHole_Pad
- removed J101: VBATG, TestPoint:TestPoint_Loop_D1.80mm_Drill1.0mm_Beaded, symbol Connector:Conn_01x01_Female
- removed J102: VBAT+, TestPoint:TestPoint_Loop_D1.80mm_Drill1.0mm_Beaded, symbol Connector:Conn_01x01_Female
- removed J103, J106: Conn_02x05_Odd_Even, Connector_PinSocket_2.54mm:PinSocket_2x05_P2.54mm_Vertical, symbol Connector_Generic:Conn_02x05_Odd_Even
- removed J104, J105, J107: Conn_02x12_Odd_Even, Connector_PinSocket_2.54mm:PinSocket_2x12_P2.54mm_Vertical, symbol Connector_Generic:Conn_02x12_Odd_Even
- removed J108: Micro_SD_Card, Connector_Card:microSD_HC_Hirose_DM3D-SF, symbol HeManTCN-rescue:Micro_SD_Card-Connector-dragonmanh7-rescue
- removed J109, J110: USB_B, Connector_USB:USB_B_OST_USB-B1HSxx_Horizontal, symbol Connector:USB_B
- removed J111: 73725-0110BLF, footprints:USB_A_Female_Vertical_RA_73725-0110BLF, symbol HeManTCN-rescue:73725-0110BLF-dk_USB-DVI-HDMI-Connectors
- removed J112: RJ45_Amphenol_RJMG1BD3B8K1ANR, Connector_RJ:RJ45_Amphenol_RJMG1BD3B8K1ANR, symbol Connector:RJ45_Amphenol_RJMG1BD3B8K1ANR
- removed J113: Screw_Terminal_01x02, Connectors_Phoenix:PhoenixContact_MC-G_02x5.08mm_Angled, symbol Connector:Screw_Terminal_01x02
- removed J114: Conn_02x03_Odd_Even, Connector_PinHeader_2.54mm:PinHeader_2x03_P2.54mm_Vertical, symbol Connector_Generic:Conn_02x03_Odd_Even
- removed J115: Conn_02x02_Odd_Even, Pin_Headers:Pin_Header_Straight_2x02_Pitch2.54mm, symbol Connector_Generic:Conn_02x02_Odd_Even
- removed J116: Screw_Terminal_01x06, Connectors_Phoenix:PhoenixContact_MC-G_06x5.08mm_Angled, symbol Connector:Screw_Terminal_01x06
- removed JP101: Jumper_2_Bridged, Jumper:SolderJumper-2_P1.3mm_Bridged_RoundedPad1.0x1.5mm, symbol Jumper:Jumper_2_Bridged
- removed JP102: BOOT, Connector_PinHeader_2.54mm:PinHeader_1x02_P2.54mm_Horizontal, symbol Device:Jumper_NC_Small
- removed L101: 68uH, Inductor_SMD:L_6.3x6.3_H3, symbol Device:L_Small
- removed R101, R102, R103, R104, R105, R106, R107, R108, R109, R110, R111, R115, R117: 4K7, Resistor_SMD:R_0805_2012Metric, symbol Device:R_Small
- removed R112: 6.49K 1%, Resistor_SMD:R_0805_2012Metric, symbol Device:R_Small
- removed R113, R114, R116: 220R, Resistor_SMD:R_0805_2012Metric, symbol Device:R_Small
- removed R118, R119: 60R, Resistor_SMD:R_0805_2012Metric, symbol Device:R_Small
- removed R120, R122: 2K2, Resistor_SMD:R_0805_2012Metric, symbol Device:R_Small
- removed R121: 120R, Resistor_SMD:R_0805_2012Metric, symbol Device:R_Small
- removed SW101: RESET, Buttons_Switches_THT:SW_Tactile_SPST_Angled_PTS645Vx31-2LFS, symbol Switch:SW_Push
- removed SW102: PC13, Buttons_Switches_THT:SW_Tactile_SPST_Angled_PTS645Vx31-2LFS, symbol Switch:SW_Push
- removed U101: STM32H743VITx, Package_QFP:LQFP-100_14x14mm_P0.5mm, symbol MCU_ST_STM32H7:STM32H743VITx
- removed U102: S25FL127SABMFI101, footprints:S25FL127SABMFI101, symbol HeManTCN-rescue:S25FL127SABMFI101-2019-03-05_02-01-41
- removed U103, U104, U105: USBLC6-2SC6, Package_TO_SOT_SMD:SOT-23-6, symbol Power_Protection:USBLC6-2SC6
- removed U106: KSZ8081RNA, Package_DFN_QFN:QFN-24-1EP_4x4mm_P0.5mm_EP2.6x2.6mm, symbol Interface_Ethernet:KSZ8081RNA
- removed U107: MIC2005A, Package_TO_SOT_SMD:SOT-23-5, symbol HeManTCN-rescue:MIC2005A-mic20xx
- removed U108: AP63203, Package_TO_SOT_SMD:TSOT-23-6, symbol HeManTCN-rescue:AP63203-reg_ap6320x
- removed U109: TCAN332, Package_TO_SOT_SMD:SOT-23-8, symbol Interface_CAN_LIN:TCAN332
- removed U110: ISL83483, Package_SO:SOIC-8_3.9x4.9mm_P1.27mm, symbol Interface_UART:ST485EBDR
- removed U111: STM32F042F6Px, Package_SO:TSSOP-20_4.4x6.5mm_P0.65mm, symbol MCU_ST_STM32F0:STM32F042F4Px
- removed U112: MVBC02D, Package_QFP:LQFP-100_14x14mm_P0.5mm, symbol MCU_ST_STM32H7:STM32H743VITx
- removed Y101: 8MHz, Crystal:Crystal_SMD_5032-2Pin_5.0x3.2mm, symbol Device:Crystal_Small
- removed Y102: 32.768KHz, Crystal:Crystal_SMD_MicroCrystal_CC7V-T1A-2Pin_3.2x1.5mm, symbol Device:Crystal_Small
- removed Y103: 25MHz, Crystal:Crystal_SMD_5032-2Pin_5.0x3.2mm, symbol Device:Crystal_Small
Connections:
- no-connect marks 8 -> 0
Other:
- note removed: "CPU"
- note removed: "DEBUG & SERIAL"
- note removed: "ETHERNET"
- note removed: "MEMORY"
- note removed: "POWER"
- note removed: "PROTOBOARD"
- note removed: "TCN - WTB"
- note removed: "USB"
- note removed: "USER INTERFACE"

Commit message: Hoja A1
Desarme las hojas jerarquicas y configure la hoja del esquematico como A1. Hay lugar suficiente (por ahora) para todo.
Parts:
- added C? (x22): 0.1u, Capacitor_SMD:C_0805_2012Metric, symbol Device:C_Small
- added C? (x3): 4.7u, Capacitor_SMD:C_0805_2012Metric, symbol Device:C_Small
- added C? (x2): 18p, Capacitor_SMD:C_0805_2012Metric, symbol Device:C_Small
- added C? (x3): 10p, Capacitor_SMD:C_0805_2012Metric, symbol Device:C_Small
- added C? (x5): 2.2u, Capacitor_SMD:C_0805_2012Metric, symbol Device:C_Small
- added C?: 10u, Capacitor_SMD:C_0805_2012Metric, symbol Device:C_Small
- added C? (x2): 22p, Capacitor_SMD:C_0805_2012Metric, symbol Device:C_Small
- added D? (x2): NUP2105L, Package_TO_SOT_SMD:SOT-23, symbol Power_Protection:NUP2105L
- added D?: LED_PC2, LED_SMD:LED_0805_2012Metric_Castellated, symbol Device:LED_Small_ALT
- added D?: LED_PWR, LED_SMD:LED_0805_2012Metric_Castellated, symbol Device:LED_Small_ALT
- added D? (x3): B120-E3, Diode_SMD:D_SOD-123, symbol Diode:B120-E3
- added H? (x4): MountingHole, MountingHole:MountingHole_3.2mm_M3_Pad_Via, symbol Mechanical:MountingHole_Pad
- added J?: VBAT+, TestPoint:TestPoint_Loop_D1.80mm_Drill1.0mm_Beaded, symbol Connector:Conn_01x01_Female
- added J?: VBATG, TestPoint:TestPoint_Loop_D1.80mm_Drill1.0mm_Beaded, symbol Connector:Conn_01x01_Female
- added J?: Micro_SD_Card, Connector_Card:microSD_HC_Hirose_DM3D-SF, symbol HeManTCN-rescue:Micro_SD_Card-Connector-dragonmanh7-rescue
- added J?: Conn_02x02_Odd_Even, Pin_Headers:Pin_Header_Straight_2x02_Pitch2.54mm, symbol Connector_Generic:Conn_02x02_Odd_Even
- added J?: Conn_02x03_Odd_Even, Connector_PinHeader_2.54mm:PinHeader_2x03_P2.54mm_Vertical, symbol Connector_Generic:Conn_02x03_Odd_Even
- added J?: Screw_Terminal_01x06, Connectors_Phoenix:PhoenixContact_MC-G_06x5.08mm_Angled, symbol Connector:Screw_Terminal_01x06
- added J? (x2): USB_B, Connector_USB:USB_B_OST_USB-B1HSxx_Horizontal, symbol Connector:USB_B
- added J?: 73725-0110BLF, footprints:USB_A_Female_Vertical_RA_73725-0110BLF, symbol HeManTCN-rescue:73725-0110BLF-dk_USB-DVI-HDMI-Connectors
- added J?: Screw_Terminal_01x02, Connectors_Phoenix:PhoenixContact_MC-G_02x5.08mm_Angled, symbol Connector:Screw_Terminal_01x02
- added J? (x3): Conn_02x12_Odd_Even, Connector_PinSocket_2.54mm:PinSocket_2x12_P2.54mm_Vertical, symbol Connector_Generic:Conn_02x12_Odd_Even
- added J? (x2): Conn_02x05_Odd_Even, Connector_PinSocket_2.54mm:PinSocket_2x05_P2.54mm_Vertical, symbol Connector_Generic:Conn_02x05_Odd_Even
- added J?: RJ45_Amphenol_RJMG1BD3B8K1ANR, Connector_RJ:RJ45_Amphenol_RJMG1BD3B8K1ANR, symbol Connector:RJ45_Amphenol_RJMG1BD3B8K1ANR
- added JP?: BOOT, Connector_PinHeader_2.54mm:PinHeader_1x02_P2.54mm_Horizontal, symbol Device:Jumper_NC_Small
- added JP?: Jumper_2_Bridged, Jumper:SolderJumper-2_P1.3mm_Bridged_RoundedPad1.0x1.5mm, symbol Jumper:Jumper_2_Bridged
- added L?: 68uH, Inductor_SMD:L_6.3x6.3_H3, symbol Device:L_Small
- added R? (x13): 4K7, Resistor_SMD:R_0805_2012Metric, symbol Device:R_Small
- added R? (x2): 2K2, Resistor_SMD:R_0805_2012Metric, symbol Device:R_Small
- added R?: 120R, Resistor_SMD:R_0805_2012Metric, symbol Device:R_Small
- added R? (x2): 60R, Resistor_SMD:R_0805_2012Metric, symbol Device:R_Small
- added R? (x3): 220R, Resistor_SMD:R_0805_2012Metric, symbol Device:R_Small
- added R?: 6.49K 1%, Resistor_SMD:R_0805_2012Metric, symbol Device:R_Small
- added SW?: RESET, Buttons_Switches_THT:SW_Tactile_SPST_Angled_PTS645Vx31-2LFS, symbol Switch:SW_Push
- added SW?: PC13, Buttons_Switches_THT:SW_Tactile_SPST_Angled_PTS645Vx31-2LFS, symbol Switch:SW_Push
- added U?: STM32H743VITx, Package_QFP:LQFP-100_14x14mm_P0.5mm, symbol MCU_ST_STM32H7:STM32H743VITx
- added U?: MVBC02D, Package_QFP:QFP-100_14x20mm_P0.5mm, symbol Bombardier:MVBC02D
- added U?: S25FL127SABMFI101, footprints:S25FL127SABMFI101, symbol HeManTCN-rescue:S25FL127SABMFI101-2019-03-05_02-01-41
- added U?: STM32F042F6Px, Package_SO:TSSOP-20_4.4x6.5mm_P0.65mm, symbol MCU_ST_STM32F0:STM32F042F4Px
- added U?: ISL83483, Package_SO:SOIC-8_3.9x4.9mm_P1.27mm, symbol Interface_UART:ST485EBDR
- added U?: TCAN332, Package_TO_SOT_SMD:SOT-23-8, symbol Interface_CAN_LIN:TCAN332
- added U? (x3): USBLC6-2SC6, Package_TO_SOT_SMD:SOT-23-6, symbol Power_Protection:USBLC6-2SC6
- added U?: MIC2005A, Package_TO_SOT_SMD:SOT-23-5, symbol HeManTCN-rescue:MIC2005A-mic20xx
- added U?: AP63203, Package_TO_SOT_SMD:TSOT-23-6, symbol HeManTCN-rescue:AP63203-reg_ap6320x
- added U?: KSZ8081RNA, Package_DFN_QFN:QFN-24-1EP_4x4mm_P0.5mm_EP2.6x2.6mm, symbol Interface_Ethernet:KSZ8081RNA
- added Y?: 8MHz, Crystal:Crystal_SMD_5032-2Pin_5.0x3.2mm, symbol Device:Crystal_Small
- added Y?: 32.768KHz, Crystal:Crystal_SMD_MicroCrystal_CC7V-T1A-2Pin_3.2x1.5mm, symbol Device:Crystal_Small
- added Y?: 25MHz, Crystal:Crystal_SMD_5032-2Pin_5.0x3.2mm, symbol Device:Crystal_Small
Connections:
- new net: C?.1, U?.73 (VCAP2)
- new net: C?.1, U?.48 (VCAP1)
- new net: C?.1, U?.13 (PH1), Y?.1
- new net: C?.1, U?.12 (PH0), Y?.2
- new net: C?.1, U?.8 (PC14), Y?.1
- new net: C?.1, U?.9 (PC15), Y?.2
- new net: C?.1, R?.1, R?.1
- new net: D?.1 (K), R?.2 (x2)
- new net: C?.1, U?.6 (BST)
- new net: C?.2, L?.1, U?.5 (SW)
- new net: D?.2 (A), J?.1 (Pin_1)
- new net: C?.1, C?.1, U?.1 (VDD_1.2)
- new net: C?.1, R?.1, U?.24 (~RST)
- new net: C?.1, U?.7 (XO), Y?.2
- new net: C?.1, U?.8 (XI), Y?.1
- new net: R?.1, U?.9 (REXT)
- new net: C?.2, J?.R4 (TCT)
- new net: C?.2, J?.R5 (RCT)
- new net: J?.L1 (LEDY_A), J?.L4 (LEDG_A), R?.1
- new net +3V3: C?.1, C?.1, C?.1, C?.1, C?.1, C?.1, C?.1, C?.1, C?.1, C?.1, C?.1, C?.1, C?.1, C?.1, C?.1, C?.1, C?.2, D?.2 (A), J?.1 (Pin_1), J?.1 (Pin_1), J?.22 (Pin_22), J?.24 (Pin_24), J?.3 (Pin_3), J?.4 (Pin_4), J?.4 (VDD), J?.5 (Pin_5), J?.6 (Pin_6), J?.7 (Pin_7), J?.9 (Pin_9), JP?.1, JP?.2 (B), L?.2, R?.1, R?.1, R?.1, R?.1, R?.1, R?.1, R?.1, R?.1, R?.2, R?.2, R?.2, R?.2, U?.1 (FB), U?.100 (VDD), U?.11 (VDD), U?.14 (VDDIO), U?.16 (VDD), U?.2 (VDDA_3.3), U?.20 (VREF+), U?.21 (VDDA), U?.27 (VDD), U?.3 (VCC), U?.5 (VDDA), U?.50 (VDD), U?.75 (VDD), U?.8 (VCC), U?.8 (VCC)
- new net +BATT: C?.1, J?.1 (Pin_1), J?.3 (Pin_3), JP?.1 (A), U?.6 (VBAT)
- new net BOOT0_B: J?.2 (Pin_2), R?.2, U?.1 (PB8)
- new net CAN_H: D?.1 (K), J?.6 (Pin_6), R?.2, U?.7 (CANH)
- new net CAN_L: D?.2 (K), J?.4 (Pin_4), R?.2, U?.6 (CANL)
- new net CAN_RX: U?.4 (RXD), U?.81 (PD0)
- new net CAN_TX: U?.1 (TXD), U?.82 (PD1)
- new net C_USBD_D+: J?.3 (D+), U?.3 (IO2)
- new net C_USBD_D-: J?.2 (D-), U?.1 (IO1)
- new net C_USBH_D+: J?.3, U?.3 (IO2)
- new net C_USBH_D-: J?.2, U?.1 (IO1)
- new net C_USB_SER_D+: J?.3 (D+), U?.3 (IO2)
- new net C_USB_SER_D-: J?.2 (D-), U?.1 (IO1)
- new net DBG_RST: C?.2, J?.4 (Pin_4), U?.4 (NRST)
- new net ENET_CRS_DV: U?.15 (CRS_DV/PHYAD[1:0]), U?.31 (PA7)
- new net ENET_MDC: R?.1, U?.11 (MDC), U?.16 (PC1)
- new net ENET_MDIO: R?.1, U?.10 (MDIO), U?.24 (PA2)
- new net ENET_REF_CLK: U?.16 (REF_CLK), U?.23 (PA1)
- new net ENET_RXD0: U?.13 (RXD0), U?.32 (PC4)
- new net ENET_RXD1: U?.12 (RXD1), U?.33 (PC5)
- new net ENET_TXD0: U?.20 (TXD0), U?.51 (PB12)
- new net ENET_TXD1: U?.21 (TXD1), U?.52 (PB13)
- new net ENET_TXEN: U?.19 (TXEN), U?.47 (PB11)
- new net ETH_LED: R?.2, U?.23 (LED0/ANEN_SPEED)
- new net GND: C?.1, C?.1, C?.1, C?.1, C?.2, C?.2, C?.2, C?.2, C?.2, C?.2, C?.2, C?.2, C?.2, C?.2, C?.2, C?.2, C?.2, C?.2, C?.2, C?.2, C?.2, C?.2, C?.2, C?.2, C?.2, C?.2, C?.2, C?.2, C?.2, C?.2, C?.2, C?.2, C?.2, C?.2, C?.2, C?.2, C?.2, D?.3 (A), D?.3 (A), H?.1, H?.1, H?.1, H?.1, J?.1 (Pin_1), J?.1 (Pin_1), J?.1 (Pin_1), J?.1 (Pin_1), J?.10 (Pin_10), J?.11 (Pin_11), J?.13 (Pin_13), J?.13 (SHIELD), J?.15 (Pin_15), J?.17 (Pin_17), J?.19 (Pin_19), J?.2 (Pin_2), J?.2 (Pin_2), J?.2 (Pin_2), J?.2 (Pin_2), J?.2 (Pin_2), J?.21 (Pin_21), J?.21 (Pin_21), J?.23 (Pin_23), J?.23 (Pin_23), J?.24 (Pin_24), J?.3 (Pin_3), J?.3 (Pin_3), J?.3 (Pin_3), J?.4, J?.4 (GND), J?.4 (GND), J?.4 (Pin_4), J?.5 (Pin_5), J?.5 (Pin_5), J?.5 (Pin_5), J?.5 (Shield), J?.5 (Shield), J?.6 (Pin_6), J?.6 (VSS), J?.7 (Pin_7), J?.7 (Pin_7), J?.8 (Pin_8), J?.9 (Pin_9), J?.9 (Pin_9), J?.9 (SHIELD), J?.L2 (LEDY_K), J?.L3 (LEDG_K), J?.R8 (GND), J?.SH, R?.1, R?.1, R?.1, R?.1, R?.1, R?.2, SW?.1, SW?.2, U?.10 (VSS), U?.15 (VSSA), U?.19 (VSSA), U?.2 (GND), U?.2 (GND), U?.2 (GND), U?.2 (GND), U?.2 (GND), U?.22 (GND), U?.25 (GND), U?.26 (VSS), U?.4 (GND), U?.4 (GND), U?.49 (VSS), U?.5 (GND), U?.74 (VSS), U?.99 (VSS)
- new net PA0: J?.10 (Pin_10), U?.22 (PA0)
- new net PA15: J?.24 (Pin_24), U?.77 (PA15)
- new net PA3: J?.12 (Pin_12), U?.25 (PA3)
- new net PA4: J?.14 (Pin_14), U?.28 (PA4)
- new net PA5: J?.16 (Pin_16), U?.29 (PA5)
- new net PA6: J?.18 (Pin_18), U?.30 (PA6)
- new net PA8: J?.4 (Pin_4), U?.67 (PA8)
- new net PB0: J?.22 (Pin_22), U?.34 (PB0)
- new net PB1: J?.20 (Pin_20), U?.35 (PB1)
- new net PB10: J?.16 (Pin_16), U?.46 (PB10)
- new net PB3: J?.17 (Pin_17), U?.89 (PB3)
- new net PB4: J?.16 (Pin_16), U?.90 (PB4)
- new net PB5: J?.15 (Pin_15), U?.91 (PB5)
- new net PB6: J?.14 (Pin_14), U?.92 (PB6)
- new net PB7: J?.13 (Pin_13), U?.93 (PB7)
- new net PB8: J?.12 (Pin_12), U?.95 (PB8)
- new net PC0: J?.4 (Pin_4), U?.15 (PC0)
- new net PC10: J?.23 (Pin_23), U?.78 (PC10)
- new net PC13: J?.2 (Pin_2), R?.2, SW?.2, U?.7 (PC13)
- new net PC2: D?.2 (A), J?.6 (Pin_6), U?.17 (PC2_C)
- new net PC3: J?.8 (Pin_8), U?.18 (PC3_C)
- new net PC6: J?.5 (Pin_5), U?.63 (PC6)
- new net PC7: J?.6 (Pin_6), U?.64 (PC7)
- new net PC9: J?.3 (Pin_3), U?.66 (PC9)
- new net PD10: J?.11 (Pin_11), U?.57 (PD10)
- new net PD11: J?.12 (Pin_12), U?.58 (PD11)
- new net PD12: J?.9 (Pin_9), U?.59 (PD12)
- new net PD13: J?.10 (Pin_10), U?.60 (PD13)
- new net PD14: J?.7 (Pin_7), U?.61 (PD14)
- new net PD15: J?.8 (Pin_8), U?.62 (PD15)
- new net PD3: J?.22 (Pin_22), U?.84 (PD3)
- new net PD4: J?.21 (Pin_21), U?.85 (PD4)
- new net PD5: J?.20 (Pin_20), U?.86 (PD5)
- new net PD6: J?.19 (Pin_19), U?.87 (PD6)
- new net PD7: J?.18 (Pin_18), U?.88 (PD7)
- new net PD8: J?.13 (Pin_13), U?.55 (PD8)
- new net PD9: J?.14 (Pin_14), U?.56 (PD9)
- new net PE11: J?.19 (Pin_19), U?.4 (~FAUKT), U?.41 (PE11)
- new net PE12: J?.20 (Pin_20), U?.3 (ENABLE), U?.42 (PE12)
- new net PE13: J?.17 (Pin_17), U?.43 (PE13)
- new net PE14: J?.18 (Pin_18), U?.44 (PE14)
- new net PE15: J?.15 (Pin_15), U?.45 (PE15)
- new net PE2: J?.11 (Pin_11), U?.1 (PE2)
- new net PE3: J?.10 (Pin_10), U?.2 (PE3)
- new net PE4: J?.9 (Pin_9), U?.3 (PE4)
- new net PE5: J?.8 (Pin_8), U?.4 (PE5)
- new net PE6: J?.7 (Pin_7), U?.5 (PE6)
- new net QSPI_IO0: U?.37 (PE7), U?.5 (SI/IO0)
- new net QSPI_IO1: U?.2 (SO/IO1), U?.38 (PE8)
- new net QSPI_IO2: U?.3 (*WP/IO2), U?.39 (PE9)
- new net QSPI_IO3: U?.40 (PE10), U?.7 (*HOLD/IO3)
- new net QSPI_SCK: U?.36 (PB2), U?.6 (CLK)
- new net RD+: J?.R3 (RD+), U?.4 (RXP)
- new net RD-: J?.R6 (RD-), U?.3 (RXM)
- new net RS485_A: D?.2 (K), J?.1 (Pin_1), R?.1, R?.2, U?.6 (A)
- new net RS485_B: D?.1 (K), J?.3 (Pin_3), R?.1, R?.2, U?.7 (B)
- new net RS485_DE: U?.2 (~RE), U?.3 (DE), U?.96 (PB9)
- new net RS485_RX: U?.1 (RO), U?.97 (PE0)
- new net RS485_TX: U?.4 (DI), U?.98 (PE1)
- new net SDMMC_CLK: J?.5 (CLK), R?.2, U?.80 (PC12)
- new net SDMMC_CMD: J?.3 (CMD), R?.2, U?.83 (PD2)
- new net SDMMC_D0: J?.7 (DAT0), R?.2, U?.65 (PC8)
- new net SDMMC_D1: J?.8 (DAT1), R?.2
- new net SDMMC_D2: J?.1 (DAT2), R?.2
- new net SDMMC_D3: J?.2 (DAT3/CD), R?.2
- new net SWCLK: J?.3 (Pin_3), U?.6 (PA0), U?.76 (PA14)
- new net SWCLK_B: J?.6 (Pin_6), U?.20 (PA14)
- new net SWDIO: J?.1 (Pin_1), U?.7 (PA1), U?.72 (PA13)
- new net SWDIO_B: J?.5 (Pin_5), U?.19 (PA13)
- new net TD+: J?.R1 (TD+), U?.6 (TXP)
- new net TD-: J?.R2 (TD-), U?.5 (TXM)
- new net U1_RX: J?.2 (Pin_2), U?.69 (PA10), U?.8 (PA2)
- new net U1_TX: J?.1 (Pin_1), U?.68 (PA9), U?.9 (PA3)
- new net USBD_D+: U?.4 (IO2), U?.71 (PA12)
- new net USBD_D-: U?.6 (IO1), U?.70 (PA11)
- new net USBH_D+: U?.4 (IO2), U?.54 (PB15)
- new net USBH_D-: U?.53 (PB14), U?.6 (IO1)
- new net USB_SER_D+: U?.18 (PA10/PA12), U?.4 (IO2)
- new net USB_SER_D-: U?.17 (PA9/PA11), U?.6 (IO1)
- new net VBUS1: D?.2 (A), J?.1 (VBUS), U?.5 (VBUS)
- new net VBUS2: D?.2 (A), J?.1 (VBUS), U?.5 (VBUS)
- new net VBUS3: C?.1, J?.1, U?.5 (VBUS), U?.5 (VOUT)
- new net VDC: C?.1, C?.1, D?.1 (K), D?.1 (K), D?.1 (K), J?.10 (Pin_10), J?.2 (Pin_2), J?.4 (Pin_4), J?.6 (Pin_6), J?.8 (Pin_8), U?.1 (VIN), U?.2 (EN), U?.3 (VIN)
- new net ~BOOT: JP?.2, R?.2, U?.94 (BOOT0)
- new net ~QSPI_CS: U?.1 (*CS), U?.79 (PC11)
- new net ~RESET: C?.1, J?.4 (Pin_4), J?.5 (Pin_5), R?.2, SW?.1, U?.10 (PA4), U?.14 (NRST)
- no-connect marks 0 -> 8
Other:
- note added: "DEBUG & SERIAL"
- note added: "MEMORY"
- note added: "POWER"
- note added: "PROTOBOARD"
- note added: "RS485 y CAN"
- note added: "USB"

Commit message: Lib IDT71V416L15PHG8
Se agregro libreria de la memoria SRAM
Parts:
- gave numbers to parts that had none: 107
Connections:
- net +3V3: now also U102.1 (VDD), U102.15 (VDD), U102.21 (VDD), U102.40 (VDD), U102.51 (VDD), U102.65 (VDD), U102.71 (VDD), U102.88 (VDD), U102.90 (VDD)
- net GND: now also U102.10 (VSS), U102.16 (VSS), U102.30 (VSS), U102.60 (VSS), U102.66 (VSS), U102.80 (VSS), U102.93 (VSS)
