File: PCB/HeManTCN/HeManTCN.sch (KiCad schematic (older format))
At the start: 112 parts, among them J101 VBATG, J102 VBAT+, J103 Micro_SD_Card, J104 Conn_02x03_Odd_Even, J105 Conn_02x02_Odd_Even, J106 Conn_02x05_Odd_Even, J107 Conn_02x12_Odd_Even, J108 Conn_02x12_Odd_Even, J109 Conn_02x05_Odd_Even, J110 Conn_02x12_Odd_Even, J111 USB_B, J112 USB_B, J113 73725-0110BLF, J114 Screw_Terminal_01x06, J115 RJ45_Amphenol_RJMG1BD3B8K1ANR, J116 Screw_Terminal_01x02, SW101 RESET, SW102 PC13, U101 STM32H743VITx, U102 MVBC02D, U103 S25FL127SABMFI101, U104 STM32F042F6Px, U105 TCAN332, U106 ISL83483, U107 USBLC6-2SC6, U108 KSZ8081RNA, U109 USBLC6-2SC6, U110 USBLC6-2SC6, U111 MIC2005A, U112 AP63203, Y101 8MHz, Y102 32.768KHz, Y103 25MHz

Commit message: VCC, GND y BusDatos
VCC y GND conectados.
BusDatos con Buffer de Datos conectado a ambos chips.
Parts:
- added unit 2 of U114
- gave numbers to parts that had none: 3
Connections:
- net labels added: DIR, MD0-MVB, MD0-u, MD1-MVB, MD1-u, MD10-MVB, MD10-u, MD11-MVB, MD11-u, MD12-MVB, MD12-u, MD13-MVB, MD13-u, MD14-MVB, MD14-u, MD15-MVB, MD15-u, MD2-MVB, MD2-u, MD3-MVB, MD3-u, MD4-MVB, MD4-u, MD5-MVB, MD5-u, MD6-MVB, MD6-u, MD7-MVB, MD7-u, MD8-MVB, MD8-u, MD9-MVB, MD9-u, OE-D_EN
- wire segments 248 -> 301
Other:
- moved on the sheet: C101, C102, C103, C104, C105, C106, C107, C108, C109, C110, C111, C112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

Commit message: Buses Trazados
Traze los Buses de Datos y Direcciones en el Esquematico para mejor comprension y analisis de las conexiones.
Parts:
- removed C126, C127: 0.1u, Capacitor_SMD:C_0805_2012Metric, symbol Device:C_Small
- removed C131: 10p, Capacitor_SMD:C_0805_2012Metric, symbol Device:C_Small
- removed D101, D102: NUP2105L, Package_TO_SOT_SMD:SOT-23, symbol Power_Protection:NUP2105L
- removed J114: Screw_Terminal_01x06, Connectors_Phoenix:PhoenixContact_MC-G_06x5.08mm_Angled, symbol Connector:Screw_Terminal_01x06
- removed R114, R116: 60R, Resistor_SMD:R_0805_2012Metric, symbol Device:R_Small
- removed R117, R119: 2K2, Resistor_SMD:R_0805_2012Metric, symbol Device:R_Small
- removed R118: 120R, Resistor_SMD:R_0805_2012Metric, symbol Device:R_Small
- removed U105: TCAN332, Package_TO_SOT_SMD:SOT-23-8, symbol Interface_CAN_LIN:TCAN332
- removed U106: ISL83483, Package_SO:SOIC-8_3.9x4.9mm_P1.27mm, symbol Interface_UART:ST485EBDR
Connections:
- net labels added: I-O, INPUT, MA1-MVB, MA1-u, MA10-MVB, MA10-u, MA11-MVB, MA11-u, MA12-MVB, MA12-u, MA13-MVB, MA13-u, MA14-MVB, MA14-u, MA15-MVB, MA15-u, MA16-MVB, MA16-u, MA17-MVB, MA18-MVB, MA2-MVB, MA2-u, MA3-MVB, MA3-u, MA4-MVB, MA4-u, MA5-MVB, MA5-u, MA6-MVB, MA6-u, MA7-MVB, MA7-u, MA8-MVB, MA8-u, MA9-MVB, MA9-u, OE-A_EN
- net labels removed: CAN_H, CAN_L, CAN_RX, CAN_TX, MA1, MA10, MA11, MA12, MA13, MA14, MA15, MA16, MA17, MA18, MA19, MA2, MA3, MA4, MA5, MA6, MA7, MA8, MA9, PB10, PC8, PD10, PD11, PD12, PD13, PD14, PD15, PD8, PD9, PE13, PE14, PE15, RS485_A, RS485_B, RS485_DE, RS485_RX, RS485_TX
- wire segments 301 -> 300
- no-connect marks 9 -> 13
Other:
- note removed: "RS485 y CAN"

Commit message: Buses Trazados en Esquematico principal
Transferi el esquematico con los buses trazados al esquematico principal. Borre algunos pines de los GPIO que no se usaran. Falta seguir borrando y chequeando.
Falta conecciones de buses al uP segun esquema dado por Martin Ribelotta.
Parts:
- removed C101: 0.1u, Capacitor_SMD:C_0805_2012Metric, symbol Device:C_Small
- removed U102: MVBC02D, Package_QFP:QFP-100_14x20mm_P0.5mm, symbol Bombardier:MVBC02D
- added C103: 0.1u, Capacitor_SMD:C_0805_2012Metric, symbol Device:C_Small
- added U104: MVBC02D, Package_QFP:QFP-100_14x20mm_P0.5mm, symbol Bombardier:MVBC02D
- IC101: Nombre (none) -> TM Memory
- U101: Nombre (none) -> uProcesador
- U102: renamed from U114; value SN74LVCR162245DGGR DataBuffer -> 74LVCR162245
- U102: renamed from U114; value SN74LVCR162245DGGR DataBuffer -> 74LVCR162245; Nombre (none) -> Data Buffer
- U103: renamed from U113; value SN74AVC16827DGVR AddressBuffer -> 74AVC16827; Nombre (none) -> Address Buffer
- renumbered C103 to C101, C120 to C116, C121 to C117, C122 to C118, C123 to C119, C124 to C120, C125 to C121, C128 to C122, C129 to C123, C132 to C124, C133 to C125, C130 to C126, C134 to C127, C135 to C128, C116 to C129, C118 to C130, C136 to C131, C137 to C132, C119 to C133, C138 to C134, C117 to C135, D103 to D101, D104 to D102, D105 to D103, D106 to D104, D107 to D105, J106 to J103, J107 to J104, J108 to J105, J115 to J106, J109 to J107, J110 to J108, J111 to J109, J112 to J110, J113 to J111, J116 to J112, J104 to J113, J105 to J114, J103 to J115, R110 to R103, R111 to R104, R112 to R105, R113 to R106, R115 to R107, R120 to R108, R103 to R109, R104 to R110, R105 to R111, R106 to R112, R107 to R113, R108 to R114, R121 to R115, R122 to R116, R109 to R117, U108 to U105, U107 to U106, U109 to U107, U110 to U108, U111 to U109, U103 to U110, U112 to U111, U104 to U112
Connections:
- net labels added: RD-MVB, RDY-MVB, TM_REQ_CPU-MVB, WR-MVB
- net labels removed: MD0, MD1, MD10, MD11, MD12, MD13, MD14, MD15, MD2, MD3, MD4, MD5, MD6, MD7, MD8, MD9, PA8, PC6, PC7, PC9
- wire segments 300 -> 451
- no-connect marks 13 -> 12
Other:
- note added: "Address Bus (1..16)"
- note added: "Data Bus (0..15)"
- note added: "Master Address Bus (1..18)"
- note added: "Master Data Bus (0..15)"
- moved on the sheet: C101, C104, C105, C107, C108, C109, C110, C111, C112, C114, C115, C116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

Commit message: Actualizacion Junio
Actualizaciones varias. uP, Docs, FMC.
Parts:
- added unit 3 of U101
- added U101?: STM32H743ZIT6, LQFP-144_STM, symbol 2020-05-20_21-53-37:STM32H743ZIT6
- added U102: 74LVCR162245, DGG48, symbol 2019-12-04_21-08-15:SN74LVCR162245DGGR
Connections:
- net labels added: PA8, PB10, PB9, PH0, PH1
- wire segments 451 -> 488
Other:
- note added: "ALIMENTACIÓN"
- note added: "FILTRADO"
- note added: "OSCILADOR PH"
- moved on the sheet: C101, C102, C103, C104, C105, C106, C107, C108, C109, C110, C111, C112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

Commit message: V 2
ERC = 0 (se corrigieron pines varios de IC en libreria).
Se cambio regulador 3,3 V por faltante en Mouser.
Se configuro correctamente FMC.
UART/USART listo.
JTAG (uP y MVBC02D) listo.
Leds actividad listo.
Parts:
- removed C132, C134: 2.2u, Capacitor_SMD:C_0805_2012Metric, symbol Device:C_Small
- removed IC101: 71V416L15PHG8, SOP80P1176X120-44N, symbol 71V416L15PHG8:71V416L15PHG8
- removed J105: Conn_02x12_Odd_Even, Connector_PinSocket_2.54mm:PinSocket_2x12_P2.54mm_Vertical, symbol Connector_Generic:Conn_02x12_Odd_Even
- removed L101: 68uH, Inductor_SMD:L_6.3x6.3_H3, symbol Device:L_Small
- removed U101: STM32H743VITx, Package_QFP:LQFP-100_14x14mm_P0.5mm, symbol MCU_ST_STM32H7:STM32H743VITx
- removed U101?: STM32H743ZIT6, LQFP-144_STM, symbol 2020-05-20_21-53-37:STM32H743ZIT6
- removed U102: 74LVCR162245, DGG48, symbol 2019-12-04_21-08-15:SN74LVCR162245DGGR
- removed U111: AP63203, Package_TO_SOT_SMD:TSOT-23-6, symbol HeManTCN-rescue:AP63203-reg_ap6320x
- added C136, C137, C138, C139, C140, C142, C143, C144, C145, C146, C148: 0.1u, Capacitor_SMD:C_0805_2012Metric, symbol Device:C_Small
- added C141: 4.7u, Capacitor_SMD:C_0805_2012Metric, symbol Device:C_Small
- added C147: 10u, Capacitor_SMD:C_0805_2012Metric, symbol Device:C_Small
- added C149, C150, C155, C156: 2.2u, Capacitor_SMD:C_0805_2012Metric, symbol Device:C_Small
- added C154: 10n, Capacitor_SMD:C_0805_2012Metric, symbol Device:C_Small
- added D106, D107, D108, D109, D110: NUP2105L, Package_TO_SOT_SMD:SOT-23, symbol Power_Protection:NUP2105L
- added D111: LED_PWR_USB, LED_SMD:LED_0805_2012Metric_Castellated, symbol Device:LED_Small_ALT
- added D112: LED_PWR_5V, LED_SMD:LED_0805_2012Metric_Castellated, symbol Device:LED_Small_ALT
- added D113: LED_USR2, LED_SMD:LED_0805_2012Metric_Castellated, symbol Device:LED_Small_ALT
- added D114: LED_uP_TM, LED_SMD:LED_0805_2012Metric_Castellated, symbol Device:LED_Small_ALT
- added D115: LED_MVB_TM, LED_SMD:LED_0805_2012Metric_Castellated, symbol Device:LED_Small_ALT
- added D116: LED_ETHERNET, LED_SMD:LED_0805_2012Metric_Castellated, symbol Device:LED_Small_ALT
- added D117: LED_SD, LED_SMD:LED_0805_2012Metric_Castellated, symbol Device:LED_Small_ALT
- added D118: LED_UART7, LED_SMD:LED_0805_2012Metric_Castellated, symbol Device:LED_Small_ALT
- added D119: LED_UART4, LED_SMD:LED_0805_2012Metric_Castellated, symbol Device:LED_Small_ALT
- added D120: LED_USART6, LED_SMD:LED_0805_2012Metric_Castellated, symbol Device:LED_Small_ALT
- added IC101: AP3512EMPTR-G1, SOIC127P600X155-9N, symbol AP3512EMPTR-G1:AP3512EMPTR-G1
- added J105: 5 VOLTS, Connector_PinSocket_2.54mm:PinSocket_2x05_P2.54mm_Vertical, symbol Connector_Generic:Conn_02x02_Odd_Even
- added J116: Screw_Terminal_01x06, Connectors_Phoenix:PhoenixContact_MC-G_06x5.08mm_Angled, symbol Connector:Screw_Terminal_01x06
- added J117: Screw_Terminal_01x03, Connectors_Phoenix:PhoenixContact_MC-G_06x5.08mm_Angled, symbol Connector:Screw_Terminal_01x03
- added J118: DB9 Hembra, Connector_Dsub:DSUB-9_Female_Horizontal_P2.77x2.84mm_EdgePinOffset4.94mm_Housed_MountingHolesOffset7.48mm, symbol TP_DCI_Gustavo_Paredes-rescue:DB9_Female-Connector
- added J119: DB9 Macho, Connector_Dsub:DSUB-9_Male_Horizontal_P2.77x2.84mm_EdgePinOffset4.94mm_Housed_MountingHolesOffset7.48mm, symbol TP_DCI_Gustavo_Paredes-rescue:DB9_Male-Connector
- added J121: JTAG MVB, Connector_PinSocket_2.54mm:PinSocket_2x05_P2.54mm_Vertical, symbol Connector_Generic:Conn_01x06
- added L102: 68uH, Inductor_SMD:L_6.3x6.3_H3, symbol Device:L_Small
- added L104: 4.7uH, Inductor_SMD:L_6.3x6.3_H3, symbol Device:L_Small
- added R118, R120, R122, R123, R125, R126, R127, R129, R130, R132: 2K2, Resistor_SMD:R_0805_2012Metric, symbol Device:R_Small
- added R119, R121, R124, R128, R131: 120R, Resistor_SMD:R_0805_2012Metric, symbol Device:R_Small
- added R133, R134, R135, R136: 10R, Resistor_SMD:R_0805_2012Metric, symbol Device:R_Small
- added R137: 10KR, Resistor_SMD:R_0805_2012Metric, symbol Device:R_Small
- added R138: 470R, Resistor_SMD:R_0805_2012Metric, symbol Device:R_Small
- added R139: 270R, Resistor_SMD:R_0805_2012Metric, symbol Device:R_Small
- added R140, R141, R142, R143, R144, R145, R146, R147: 220R, Resistor_SMD:R_0805_2012Metric, symbol Device:R_Small
- added R148: 4K7, Resistor_SMD:R_0805_2012Metric, symbol Device:R_Small
- added R149, R151: 10K, Resistor_SMD:R_0805_2012Metric, symbol Device:R_Small
- added R150: 100K, Resistor_SMD:R_0805_2012Metric, symbol Device:R_Small
- added R152: 18K, Resistor_SMD:R_0805_2012Metric, symbol Device:R_Small
- added R153: 8.2K, Resistor_SMD:R_0805_2012Metric, symbol Device:R_Small
- added SW103: RESET_MVB, Buttons_Switches_THT:SW_Tactile_SPST_Angled_PTS645Vx31-2LFS, symbol Switch:SW_Push
- added SW104: SWITCH MVB, symbol Switch:SW_DIP_x04
- added SW105: USER_SWITCH2, Buttons_Switches_THT:SW_Tactile_SPST_Angled_PTS645Vx31-2LFS, symbol Switch:SW_Push
- added unit 2 of U101
- added U113: CY7C1051DV33-10ZSXI, TSOP-44, symbol CY7C1051DV33-10ZSXI:CY7C1051DV33-10ZSXI
- added U114, U115, U116, U117, U118: ISL83485IBZ, SOIC8_4X5_INR, symbol 2020-07-16_16-51-34:ISL83485IBZ
- added U119: AP63205WU-7, SOIC_05WU-7_DIO, symbol 2020-07-16_18-36-02:AP63205WU-7
- added Y104: SG7050CAN_24.000000M-TJGA3, SG7050CAN1000000MTJGA3, symbol SG7050CAN_24.000000M-TJGA3:SG7050CAN_24.000000M-TJGA3
- C131: value 0.1u -> 3.3n; manf# 885012207098 -> CL21B225KPFNNNE
- D104: value LED_PWR -> LED_PWR_3,3V
- D105: value LED_PC2 -> LED_USR1
- J103: value Conn_02x05_Odd_Even -> 12 VOLTS; symbol Connector_Generic:Conn_02x05_Odd_Even -> Connector_Generic:Conn_02x02_Odd_Even
- J104: value Conn_02x12_Odd_Even -> Conn_02x10_Odd_Even; symbol Connector_Generic:Conn_02x12_Odd_Even -> Connector_Generic:Conn_02x10_Odd_Even
- J107: value Conn_02x05_Odd_Even -> 3,3 VOLTS; symbol Connector_Generic:Conn_02x05_Odd_Even -> Connector_Generic:Conn_02x02_Odd_Even
- J108: value Conn_02x12_Odd_Even -> Conn_02x07_Odd_Even; symbol Connector_Generic:Conn_02x12_Odd_Even -> Connector_Generic:Conn_02x07_Odd_Even
- J114: value Conn_02x02_Odd_Even -> JTAG uP
- SW102: value PC13 -> USER_SWITCH1
Connections:
- net labels added: +12V, +5V, CLK_MVB, DATA_ACK_MVB, ENABLE_USB, ERR_USB, GNDPWR, GPIO_ANALOG1, GPIO_ANALOG2, GPIO_ANALOG3, GPIO_IN1, GPIO_IN2, GPIO_IN3, GPIO_IN4, GPIO_IN5, GPIO_IN6, GPIO_OUT1, GPIO_OUT2, GPIO_OUT3, GPIO_OUT4, GPIO_OUT5, GPIO_OUT6, INT0_EXT_MVB, INT0_MVB, INT1_EXT_MVB, INT1_MVB, INT2_EXT_MVB, INT3_EXT_MVB, JTAG_MVB_TCK, JTAG_MVB_TDI, JTAG_MVB_TDO, JTAG_MVB_TMS, JTAG_MVB_TRST, LED_ETHERNET, LED_MVB_TM, LED_SD, LED_UART4, LED_UART7, LED_USART6, LED_USR1, LED_USR2, LED_uP_TM, MA17-u, MA18-u, MA19-MVB, MA19-u, MVB485_A1, MVB485_A2, MVB485_B1, MVB485_B2, MVB485_ENA, MVB485_ICA, MVB485_ICB, MVB485_OUT, PC14-OSC32_IN, PC15-OSC32_OUT, PH0-OSC_IN, PH1-OSC_OUT, RESET_MVB, RS485_A1, RS485_A2, RS485_A3, RS485_B1, RS485_B2, RS485_B3, SCAN_EN_MVB, SCAN_TEST_MVB, STROBE_MVB, TMR1, TMR2, UART4_DE, UART4_RX, UART4_TX, UART7_DE, UART7_RX, UART7_TX, USART3_RX, USART3_TX, USART6_DE, USART6_RX, USART6_TX, USB_OTG_FS_DM, USB_OTG_FS_DP, USB_OTG_HS_DM, USB_OTG_HS_DP, USER_SWITCH1, USER_SWITCH2, Z-MODE_MVB
- net labels removed: I-O, INPUT, PA0, PA15, PA3, PA4, PA5, PA6, PA8, PB0, PB1, PB10, PB3, PB4, PB5, PB6, PB7, PB8, PB9, PC0, PC10, PC13, PC2, PC3, PD3, PD4, PD5, PD6, PD7, PE11, PE12, PE2, PE3, PE4, PE5, PE6, PH0, PH1, U1_RX, U1_TX, USBD_D+, USBD_D-, USBH_D+, USBH_D-
- wire segments 488 -> 489
- no-connect marks 12 -> 14
Other:
- note added: "A. Bus_5V"
- note added: "A. Bus_GND"
- note added: "A. Data_N"
- note added: "A. Data_P"
- note added: "ALIMENTACIÓN BATERÍA"
- note added: "ALIMENTACIÓN C.I."
- note added: "B. Bus_5V"
- note added: "B. Bus_GND"
- note added: "B. Data_N"
- note added: "B. Data_P"
- note added: "Connection acc.: IEC61375-3"
- note added: "ETHERNET"
- note added: "FILTRADO 3,3 V"
- note added: "FILTRADO 5 V"
- note added: "LEDS"
- note added: "MEMORY SD"
- note added: "MVB (RS-485)"
- note added: "MVB PORT RS485"
- note added: "OSCILADOR MVB"
- note added: "OSCILADOR RTC uP"
- note added: "OSCILADOR uP"
- note added: "POWER 3,3 V"
- note added: "POWER 3,3 V y 5 V"
- note added: "POWER 5 V"
- note added: "PROCESADOR y MVB"
- note added: "PULSADORES"
- note added: "SWITCHS"
- note added: "UART uP (RS-485)"
- note added: "USART uP (RS-485)"
- note removed: "ALIMENTACIÓN"
- note removed: "Address Bus (1..16)"
- note removed: "Data Bus (0..15)"
- note removed: "FILTRADO"
- note removed: "MEMORY"
- note removed: "Master Address Bus (1..18)"
- note removed: "Master Data Bus (0..15)"
- note removed: "OSCILADOR PH"
- note removed: "POWER"
- moved on the sheet: C102, C103, C104, C105, C106, C107, C113, C115, C116, C117, C118, C119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

Commit message: Carpeta Lib/Foot/3D
Se creo carpeta de librerias/huellas y 3D.
Parts:
- removed LOGO101: Logo_Open_Hardware_Small, footprints:ciaa_7-logo, symbol Graphic:Logo_Open_Hardware_Small
- removed LOGO102: Logo_Open_Hardware_Small, footprints:unqui-logo, symbol Graphic:Logo_Open_Hardware_Small
- U101: symbol 2020-05-20_21-53-37:STM32H743ZIT6 -> HeManTCN-rescue:STM32H743ZIT6-2020-05-20_21-53-37
- U106, U107, U108: symbol Power_Protection:USBLC6-2SC6 -> HeManTCN-rescue:USBLC6-2SC6-Power_Protection
- U112: symbol MCU_ST_STM32F0:STM32F042F4Px -> HeManTCN-rescue:STM32F042F4Px-MCU_ST_STM32F0
Changed lines of the file:
@@
 $EndDescr
 $Comp
-L Graphic:Logo_Open_Hardware_Small LOGO101
-U 1 1 5E3428D1
-P 29500 19350
-F 0 "LOGO101" H 29500 19625 50  0001 C CNN
-F 1 "Logo_Open_Hardware_Small" H 29500 19125 50  0001 C CNN
-F 2 "footprints:ciaa_7-logo" H 29500 19350 50  0001 C CNN
-F 3 "~" H 29500 19350 50  0001 C CNN
-	1    29500 19350
-	1    0    0    -1
-$EndComp
-$Comp
-L Graphic:Logo_Open_Hardware_Small LOGO102
-U 1 1 5E3428D2
-P 30200 19350
-F 0 "LOGO102" H 30200 19625 50  0001 C CNN
-F 1 "Logo_Open_Hardware_Small" H 30200 19125 50  0001 C CNN
-F 2 "footprints:unqui-logo" H 30200 19350 50  0001 C CNN
-F 3 "~" H 30200 19350 50  0001 C CNN
-	1    30200 19350
-	1    0    0    -1
-$EndComp
-$Comp
 L power:GND #PWR0104
 U 1 1 5DA6482C
@@
 DEBUG & SERIAL
 $Comp
-L MCU_ST_STM32F0:STM32F042F4Px U112
+L HeManTCN-rescue:STM32F042F4Px-MCU_ST_STM32F0 U112
 U 1 1 5DA6F3C2
 P 24150 12300
@@
 USB_SER_D-
 $Comp
-L Power_Protection:USBLC6-2SC6 U107
+L HeManTCN-rescue:USBLC6-2SC6-Power_Protection U107
 U 1 1 5DA7B096
 P 18350 2550
@@
 $EndComp
 $Comp
-L Power_Protection:USBLC6-2SC6 U108
+L HeManTCN-rescue:USBLC6-2SC6-Power_Protection U108
 U 1 1 5DA7B09E
 P 18350 3800
@@
 $EndComp
 $Comp
-L Power_Protection:USBLC6-2SC6 U106
+L HeManTCN-rescue:USBLC6-2SC6-Power_Protection U106
 U 1 1 5DA7B0A6
 P 18300 5000
@@
 TM_REQ_CPU-MVB
 $Comp
-L 2020-05-20_21-53-37:STM32H743ZIT6 U101
+L HeManTCN-rescue:STM32H743ZIT6-2020-05-20_21-53-37 U101
 U 1 1 5ECD5F3F
 P 2650 12000
@@
 $EndComp
 $Comp
-L 2020-05-20_21-53-37:STM32H743ZIT6 U101
+L HeManTCN-rescue:STM32H743ZIT6-2020-05-20_21-53-37 U101
 U 3 1 5ECC2AF4
 P 2700 3500
@@
 $EndComp
 $Comp
-L 2020-05-20_21-53-37:STM32H743ZIT6 U101
+L HeManTCN-rescue:STM32H743ZIT6-2020-05-20_21-53-37 U101
 U 2 1 5F253D72
 P 2950 8250

Commit message: Huellas V1
Se actualizaron algunas huellas.
Parts:
- IC101: value AP3512EMPTR-G1 -> IC Reg 3,3 V AP3512EMPTR-G1; footprint SOIC127P600X155-9N -> footprintsSnifferTCN:AP3512EMPTR-G1
- J104: value Conn_02x10_Odd_Even -> Protoboard GPIO 1
- J106: value RJ45_Amphenol_RJMG1BD3B8K1ANR -> Conector RJ45
- J108: value Conn_02x07_Odd_Even -> Protoboard GPIO 2
- J109: value USB_B -> Conector USB_B 2
- J110: value USB_B -> Conector USB_B 1
- J111: value 73725-0110BLF -> Conector USB Vertical; footprint footprints:USB_A_Female_Vertical_RA_73725-0110BLF -> footprintsSnifferTCN:USB_A_Female_Vertical_RA_73725-0110BLF
- J112: value Screw_Terminal_01x02 -> Conector 12 V/GND x 2; footprint Connectors_Phoenix:PhoenixContact_MC-G_02x5.08mm_Angled -> footprintsSnifferTCN:Bornera2Pines_282837-2
- J113: value Conn_02x03_Odd_Even -> Debug/Serial
- J114: footprint Pin_Headers:Pin_Header_Straight_2x02_Pitch2.54mm -> Connector_PinHeader_2.54mm:PinHeader_2x02_P2.54mm_Vertical
- J116: value Screw_Terminal_01x06 -> Conector RS485 x 6; footprint Connectors_Phoenix:PhoenixContact_MC-G_06x5.08mm_Angled -> footprintsSnifferTCN:Bornera6Pines_282837-6
- J117: value Screw_Terminal_01x03 -> Conector RS485 x 3; footprint Connectors_Phoenix:PhoenixContact_MC-G_06x5.08mm_Angled -> footprintsSnifferTCN:Bornera3Pines_282837-3
- JP101: footprint Jumper:SolderJumper-2_P1.3mm_Bridged_RoundedPad1.0x1.5mm -> Connector_PinHeader_2.54mm:PinHeader_1x02_P2.54mm_Vertical
- SW102: value USER_SWITCH1 -> Pulsador 1
- SW105: value USER_SWITCH2 -> Pulsador 2
- U101: value STM32H743ZIT6 -> IC uP STM32H743ZIT6
- U102: value 74LVCR162245 -> IC DB 74LVCR162245
- U105: value KSZ8081RNA -> IC Ethernet KSZ8081RNA
- U106, U107, U108: value USBLC6-2SC6 -> IC USBLC6-2SC6
- U112: value STM32F042F6Px -> IC Debug/Serial
- U113: value CY7C1051DV33-10ZSXI -> IC TM CY7C1051DV33-10ZSXI
- U114, U115, U116, U117, U118: value ISL83485IBZ -> IC RS485 ISL83485IBZ
- U119: value AP63205WU-7 -> IC Reg 5 V AP63205WU-7
- Y104: value SG7050CAN_24.000000M-TJGA3 -> XT 24 MHz; footprint SG7050CAN1000000MTJGA3 -> footprintsSnifferTCN:SG7050CAN1000000MTJGA3

Commit message: WIP
Renombrado .ioc a FirmwareSnifferTCN.ioc
Check hasta pin 37 uP entre .ioc y esquematico.
Parts:
- JP101: value Jumper_2_Bridged -> Jumper1
- SW101, SW102, SW103, SW105: footprint Buttons_Switches_THT:SW_Tactile_SPST_Angled_PTS645Vx31-2LFS -> footprintsSnifferTCN:Pulsador_TL3342F160QG
- SW104: footprint (none) -> footprintsSnifferTCN:Pulsador_TL3342F160QG
- U102: footprint DGG48 -> footprintsSnifferTCN:DataBuffer SN74LVCR162245DGGR
- U103: footprint DGV56 -> footprintsSnifferTCN:AddressBuffer SN74AVC16827DGVR
- U104: footprint Package_QFP:QFP-100_14x20mm_P0.5mm -> Package_QFP:PQFP-100_14x20mm_P0.65mm
Connections:
- net PH0-OSC_IN: no longer U101.23 (PH0-OSC_IN)
- net PH1-OSC_OUT: no longer U101.24 (PH1-OSC_OUT)
- net PC14-OSC32_IN renamed RCC-OSC32_IN
- net PC15-OSC32_OUT renamed RCC-OSC32_OUT
- new net RCC-OSC_IN: U101.23 (PH0-OSC_IN)
- new net RCC-OSC_OUT: U101.24 (PH1-OSC_OUT)
Changed lines of the file:
@@
 AR Path="/5DA2C15A/5DA64962" Ref="JP?"  Part="1"
 F 0 "JP101" V 1250 1600 50  0000 R CNN
-F 1 "Jumper_2_Bridged" H 1650 1750 50  0000 R CNN
+F 1 "Jumper1" H 1450 1750 50  0000 R CNN
 F 2 "Connector_PinHeader_2.54mm:PinHeader_1x02_P2.54mm_Vertical" H 1300 1650 50  0001 C CNN
 F 3 "~" H 1300 1650 50  0001 C CNN
@@
 F 0 "SW101" V 22496 2202 50  0000 R CNN
 F 1 "RESET" H 22450 2050 50  0000 R CNN
-F 2 "Buttons_Switches_THT:SW_Tactile_SPST_Angled_PTS645Vx31-2LFS" H 22450 2450 50  0001 C CNN
+F 2 "footprintsSnifferTCN:Pulsador_TL3342F160QG" H 22450 2450 50  0001 C CNN
 F 3 "~" H 22450 2450 50  0001 C CNN
 F 4 "TL3342" H 13650 950 50  0001 C CNN "manf#"
@@
 F 0 "SW102" V 23396 2202 50  0000 R CNN
 F 1 "Pulsador 1" V 23305 2202 50  0000 R CNN
-F 2 "Buttons_Switches_THT:SW_Tactile_SPST_Angled_PTS645Vx31-2LFS" H 23350 2450 50  0001 C CNN
+F 2 "footprintsSnifferTCN:Pulsador_TL3342F160QG" H 23350 2450 50  0001 C CNN
 F 3 "~" H 23350 2450 50  0001 C CNN
 F 4 "PTS645VM31-2 LFS" H 14100 950 50  0001 C CNN "manf#"
@@
 F 0 "U102" H 8600 7200 60  0000 C CNB
 F 1 "IC DB 74LVCR162245" H 8550 6800 60  0000 C CNB
-F 2 "DGG48" H 8600 8340 60  0001 C CNN
+F 2 "footprintsSnifferTCN:DataBuffer SN74LVCR162245DGGR" H 8600 8340 60  0001 C CNN
 F 3 "" H 7800 8100 60  0000 C CNN
 F 4 "Data Buffer" H 8600 5900 79  0000 C CNB "Nombre"
@@
 F 0 "U102" H 6500 2600 60  0000 C CNB
 F 1 "IC DB 74LVCR162245" H 6500 3450 60  0000 C CNB
-F 2 "DGG48" H 6500 3740 60  0001 C CNN
+F 2 "footprintsSnifferTCN:DataBuffer SN74LVCR162245DGGR" H 6500 3740 60  0001 C CNN
 F 3 "" H 5700 3500 60  0000 C CNN
 F 4 "Data Buffer" H 6500 1400 79  0000 C CNB "Nombre"
@@
 Connection ~ 7400 3800
 Text Label 5250 12100 0    50   ~ 0
-PH1-OSC_OUT
+RCC-OSC_OUT
 Wire Notes Line
 	2100 2150 2100 1450
@@
 USER_SWITCH1
 Text Label 5250 15400 0    50   ~ 0
-PC14-OSC32_IN
+RCC-OSC32_IN
 Text Label 5250 12000 0    50   ~ 0
-PC15-OSC32_OUT
+RCC-OSC32_OUT
 Text Label 2650 14100 2    50   ~ 0
 MD2-u
@@
 MD1-u
 Text Label 4750 1550 2    50   ~ 0
-PC14-OSC32_IN
+RCC-OSC32_IN
 Text Label 4750 1650 2    50   ~ 0
-PC15-OSC32_OUT
+RCC-OSC32_OUT
 Wire Notes Line
 	4000 2200 4000 1450
@@
 F 0 "U103" H 8600 9950 60  0000 C CNB
 F 1 "74AVC16827" H 8600 9650 51  0000 C CNN
-F 2 "DGV56" H 8600 10990 60  0001 C CNN
+F 2 "footprintsSnifferTCN:AddressBuffer SN74AVC16827DGVR" H 8600 10990 60  0001 C CNN
 F 3 "" H 7300 10750 60  0000 C CNN
 F 4 "Address Buffer" H 8600 9150 79  0000 C CNB "Nombre"
@@
 F 0 "U104" H 12400 12750 62  0000 C CNB
 F 1 "MVBC02D" H 12400 12300 100 0000 C CNN
-F 2 "Package_QFP:QFP-100_14x20mm_P0.5mm" H 11600 9650 50  0001 R CNN
+F 2 "Package_QFP:PQFP-100_14x20mm_P0.65mm" H 11600 9650 50  0001 R CNN
 F 3 "TEXTO" H 11700 15250 50  0001 C CNN
 F 4 "MVB" H 12400 12000 79  0000 C CNB "Nombre"
@@
 F 0 "SW103" V 23046 2202 50  0000 R CNN
 F 1 "RESET_MVB" H 23000 2050 50  0000 R CNN
-F 2 "Buttons_Switches_THT:SW_Tactile_SPST_Angled_PTS645Vx31-2LFS" H 23000 2450 50  0001 C CNN
+F 2 "footprintsSnifferTCN:Pulsador_TL3342F160QG" H 23000 2450 50  0001 C CNN
 F 3 "~" H 23000 2450 50  0001 C CNN
 F 4 "TL3342" H 14200 950 50  0001 C CNN "manf#"
@@
 F 0 "SW104" H 25750 2850 50  0000 C CNN
 F 1 "SWITCH MVB" H 25750 2750 50  0000 C CNN
-F 2 "" H 25750 2350 50  0001 C CNN
+F 2 "footprintsSnifferTCN:Pulsador_TL3342F160QG" H 25750 2350 50  0001 C CNN
 F 3 "" H 25750 2350 50  0001 C CNN
 	1    25750 2350
@@
 VBUS1
 Text Label 2950 9850 2    50   ~ 0
-PH0-OSC_IN
+RCC-OSC_IN
 Text Label 2650 13100 2    50   ~ 0
 LED_USR1
@@
 F 0 "SW105" V 23996 2202 50  0000 R CNN
 F 1 "Pulsador 2" V 23905 2202 50  0000 R CNN
-F 2 "Buttons_Switches_THT:SW_Tactile_SPST_Angled_PTS645Vx31-2LFS" H 23950 2450 50  0001 C CNN
+F 2 "footprintsSnifferTCN:Pulsador_TL3342F160QG" H 23950 2450 50  0001 C CNN
 F 3 "~" H 23950 2450 50  0001 C CNN
 F 4 "PTS645VM31-2 LFS" H 14700 950 50  0001 C CNN "manf#"
